File: motordriver-2x.sch (KiCad schematic (older format))
At the start: 397 parts

Commit message: start connecting pins
Connections:
- net ENCA1: now also U?.41 (ADC1_IN5/ADC2_IN5/DAC_OUT2/SPI1_SCK/TIM2_CH1/TIM2_ETR/TIM8_CH1N/USB_OTG_HS_ULPI_CK/PA5)
- net ENCA2: now also U?.81 (FMC_A17/FMC_ALE/TIM4_CH1/USART3_RTS/PD12)
- net ENCB1: now also U?.133 (I2S3_CK/SPI1_SCK/SPI3_SCK/SYS_JTDO-SWO/TIM2_CH2/PB3)
- net ENCB2: now also U?.82 (FMC_A18/TIM4_CH2/PD13)
- net HALL_A1: now also U?.134 (I2S3_ext_SD/SPI1_MISO/SPI3_MISO/SYS_JTRST/TIM3_CH1/PB4); no longer D?.1, R?.1, R?.2
- net HALL_B1: now also U?.135 (CAN2_RX/DCMI_D10/ETH_PPS_OUT/FMC_SDCKE1/I2C1_SMBA/I2S3_SD/SPI1_MOSI/SPI3_MOSI/TIM3_CH2/USB_OTG_HS_ULPI_D7/PB5); no longer D?.2, R?.1, R?.2
- net HALL_C1: now also U?.136 (CAN2_TX/DCMI_D5/FMC_SDNE1/I2C1_SCL/TIM4_CH1/USART1_TX/PB6); no longer D?.4, R?.1, R?.2
- net INHA1: now also U?.60 (PE9/DAC_EXTI9/FMC_D6/FMC_DA6/TIM1_CH1)
- net INHA2: now also U?.96 (DCMI_D0/I2S2_MCK/LTDC_HSYNC/SDIO_D6/TIM3_CH1/TIM8_CH1/USART6_TX/PC6)
- net INHB1: now also U?.64 (PE11/ADC1_EXTI11/ADC2_EXTI11/ADC3_EXTI11/FMC_D8/FMC_DA8/LTDC_G3/SPI4_NSS/TIM1_CH2)
- net INHB2: now also U?.97 (DCMI_D1/I2S3_MCK/LTDC_G6/SDIO_D7/TIM3_CH2/TIM8_CH2/USART6_RX/PC7)
- net INHC1: now also U?.66 (PE13/FMC_D10/FMC_DA10/LTDC_DE/SPI4_MISO/TIM1_CH3)
- net INHC2: now also U?.98 (DCMI_D2/SDIO_D0/TIM3_CH3/TIM8_CH3/USART6_CK/PC8)
- net INLA1: now also U?.59 (PE8/FMC_D5/FMC_DA5/TIM1_CH1N/UART7_TX)
- net INLA2: now also U?.43 (ADC1_IN7/ADC2_IN7/ETH_CRS_DV/ETH_RX_DV/SPI1_MOSI/TIM14_CH1/TIM1_CH1N/TIM3_CH2/TIM8_CH1N/PA7)
- net INLB1: now also U?.63 (PE10/FMC_D7/FMC_DA7/TIM1_CH2N)
- net INLB2: now also U?.75 (I2S2_ext_SD/SPI2_MISO/TIM12_CH1/TIM1_CH2N/TIM8_CH2N/USART3_RTS/USB_OTG_HS_DM/PB14)
- net INLC1: now also U?.65 (PE12/FMC_D9/FMC_DA9/LTDC_B4/SPI4_SCK/TIM1_CH3N)
- net INLC2: now also U?.76 (ADC1_EXTI15/ADC2_EXTI15/ADC3_EXTI15/I2S2_SD/RTC_REFIN/SPI2_MOSI/TIM12_CH2/TIM1_CH3N/TIM8_CH3N/USB_OTG_HS_DP/PB15)
- net SWO: no longer U?.133 (I2S3_CK/SPI1_SCK/SPI3_SCK/SYS_JTDO-SWO/TIM2_CH2/PB3)
- net HALL_A2: now reaches U?.34 (ADC1_IN0/ADC2_IN0/ADC3_IN0/ETH_CRS/SYS_WKUP/TIM2_CH1/TIM2_ETR/TIM5_CH1/TIM8_ETR/UART4_TX/USART2_CTS/PA0)
- net HALL_A2: now also D?.1, R?.1, R?.2
- net HALL_B2: now reaches U?.35 (ADC1_IN1/ADC2_IN1/ADC3_IN1/ETH_REF_CLK/ETH_RX_CLK/TIM2_CH2/TIM5_CH2/UART4_RX/USART2_RTS/PA1)
- net HALL_B2: now also D?.2, R?.1, R?.2
- net HALL_C2: now reaches U?.36 (ADC1_IN2/ADC2_IN2/ADC3_IN2/ETH_MDIO/TIM2_CH3/TIM5_CH3/TIM9_CH1/USART2_TX/PA2)
- net HALL_C2: now also D?.4, R?.1, R?.2
Other:
- note added: "Add current sensing to each supply"
- note added: "Investigate up to vcc-2v input range\nConsider TLV2401 or TLV2474 instead\nAdd clipping diodes to output"
Changed lines of the file:
@@
 Text GLabel 11575 3250 2    50   Input ~ 0
 UART1_RX
-Text GLabel 11575 4250 2    50   Input ~ 0
+Text GLabel 12350 3800 2    50   Input ~ 0
 SWO
 $Comp
@@
 Connection ~ 25975 11125
 Text GLabel 25925 11125 0    50   Input ~ 0
-HALL_A1
+HALL_A2
 Text GLabel 25925 11225 0    50   Input ~ 0
-HALL_B1
+HALL_B2
 Text GLabel 25925 11325 0    50   Input ~ 0
-HALL_C1
+HALL_C2
 $Comp
 L SwEmb:D_TPD3E001 D?
@@
 U 1 1 806F3944
 P 3400 15900
-F 0 "U?" H 3428 16367 50  0000 C CNN
-F 1 "IC_TPS54360DDA" H 3428 16276 50  0000 C CNN
+F 0 "U?" H 3425 16375 50  0000 C CNN
+F 1 "IC_TPS54360DDA" H 3425 16300 50  0000 C CNN
 F 2 "SOIC:SOIC127P600X175_HS-9N" H 3450 15450 50  0001 L CIN
 F 3 "" H 3400 15900 50  0001 C CNN
@@
 Text GLabel 14075 3325 0    50   Input ~ 0
 ENCOC2
-Text GLabel 14075 3525 0    50   Input ~ 0
+Text GLabel 11575 2750 2    50   Input ~ 0
 ENCA1
 Text GLabel 14075 3625 0    50   Input ~ 0
 ENCAF1
-Text GLabel 14075 3825 0    50   Input ~ 0
+Text GLabel 11575 4250 2    50   Input ~ 0
 ENCB1
 Text GLabel 14075 3925 0    50   Input ~ 0
@@
 Text GLabel 14075 5925 0    50   Input ~ 0
 EN_GATE1
-Text GLabel 14075 6025 0    50   Input ~ 0
-INHA1
-Text GLabel 14075 6125 0    50   Input ~ 0
+Text GLabel 2375 8150 0    50   Input ~ 0
 INLA1
-Text GLabel 14075 6225 0    50   Input ~ 0
+Text GLabel 2375 8450 0    50   Input ~ 0
 INHB1
-Text GLabel 14075 6325 0    50   Input ~ 0
+Text GLabel 2375 8350 0    50   Input ~ 0
 INLB1
-Text GLabel 14075 6425 0    50   Input ~ 0
+Text GLabel 2375 8650 0    50   Input ~ 0
 INHC1
-Text GLabel 14075 6525 0    50   Input ~ 0
+Text GLabel 2375 8550 0    50   Input ~ 0
 INLC1
 Text GLabel 14075 6625 0    50   Input ~ 0
@@
 Text GLabel 14075 7025 0    50   Input ~ 0
 VSC1
-Text GLabel 14075 7725 0    50   Input ~ 0
+Text GLabel 11575 8550 2    50   Input ~ 0
 ENCA2
 Text GLabel 14075 7825 0    50   Input ~ 0
 ENCAF2
-Text GLabel 14075 8025 0    50   Input ~ 0
+Text GLabel 11575 8650 2    50   Input ~ 0
 ENCB2
 Text GLabel 14075 8125 0    50   Input ~ 0
@@
 Text GLabel 14075 10125 0    50   Input ~ 0
 EN_GATE2
-Text GLabel 14075 10225 0    50   Input ~ 0
+Text GLabel 11575 6250 2    50   Input ~ 0
 INHA2
-Text GLabel 14075 10325 0    50   Input ~ 0
+Text GLabel 11575 2950 2    50   Input ~ 0
 INLA2
-Text GLabel 14075 10425 0    50   Input ~ 0
+Text GLabel 11575 6350 2    50   Input ~ 0
 INHB2
-Text GLabel 14075 10525 0    50   Input ~ 0
+Text GLabel 11575 5350 2    50   Input ~ 0
 INLB2
-Text GLabel 14075 10625 0    50   Input ~ 0
+Text GLabel 11575 6450 2    50   Input ~ 0
 INHC2
-Text GLabel 14075 10725 0    50   Input ~ 0
+Text GLabel 11575 5450 2    50   Input ~ 0
 INLC2
 Text GLabel 14075 10825 0    50   Input ~ 0
@@
 Text GLabel 14075 11425 0    50   Input ~ 0
 VSC2
-Text GLabel 14075 7125 0    50   Input ~ 0
+Text GLabel 11575 4350 2    50   Input ~ 0
 HALL_A1
-Text GLabel 14075 7225 0    50   Input ~ 0
+Text GLabel 11575 4450 2    50   Input ~ 0
 HALL_B1
-Text GLabel 14075 7325 0    50   Input ~ 0
-HALL_C1
-Text GLabel 14075 11525 0    50   Input ~ 0
-HALL_A1
-Text GLabel 14075 11625 0    50   Input ~ 0
-HALL_B1
-Text GLabel 14075 11725 0    50   Input ~ 0
+Text GLabel 11575 4550 2    50   Input ~ 0
 HALL_C1
+Text GLabel 11575 2250 2    50   Input ~ 0
+HALL_A2
+Text GLabel 11575 2350 2    50   Input ~ 0
+HALL_B2
+Text GLabel 11575 2450 2    50   Input ~ 0
+HALL_C2
 Text GLabel 13000 9775 2    50   Input ~ 0
 POT1
@@
 Text Notes 2675 22350 0    39   ~ 0
 Add possibility to bypass
+Text Notes 7825 15225 0    39   ~ 0
+Add current sensing to each supply
+Text Notes 3200 17250 0    39   ~ 0
+Investigate up to vcc-2v input range\nConsider TLV2401 or TLV2474 instead\nAdd clipping diodes to output
+Text GLabel 2375 8250 0    50   Input ~ 0
+INHA1
 $EndSCHEMATC

Commit message: connect more pins to mcu, change opamp and add analog multiplexer
Parts:
- added C?: CAP_100nF_50V_0402, Capacitor_SMD:C_0402_1005Metric, symbol SwEmb:CAP_100nF_50V_0402
- added D? (x8): D_BAT54S, Package_TO_SOT_SMD:SOT-23, symbol SwEmb:D_BAT54S
- added R? (x8): RES_0R_0402, Resistor_SMD:R_0402_1005Metric, symbol SwEmb:RES_0R_0402
- added U?: IC_SN74LV4051, Package_SO:TSSOP-16_4.4x5mm_P0.65mm, symbol SwEmb:IC_SN74LV4051
- U? (x8): value IC_LM324 -> IC_TLV2474; symbol SwEmb:IC_LM324 -> SwEmb:IC_TLV2474; MPN LM324D -> TLV2474CDR
Connections:
- net ENCMISO2 is gone; now on net ENCMISO1: U?.3 (~D3FAULT/SDO)
- net ENCMOSI2 is gone; now on net ENCMOSI1: U?.6 (TTL/SDI)
- net ENCSCK2 is gone; now on net ENCSCK1: U?.5 (SNGL/SCK)
- net AIN_VDD_5V: now also D?.2, D?.2, D?.2, D?.2, D?.2, D?.2, D?.2, D?.2
- net CANFD_MISO: now also U?.127 (PG12/FMC_NE4/LTDC_B1/LTDC_B4/SPI6_MISO/USART6_RTS)
- net CANFD_MOSI: now also U?.129 (PG14/ETH_TXD1/FMC_A25/SPI6_MOSI/USART6_TX)
- net CANFD_SCK: now also U?.128 (PG13/ETH_TXD0/FMC_A24/SPI6_SCK/USART6_CTS)
- net ENCMISO1: now also U?.112 (ADC1_EXTI11/ADC2_EXTI11/ADC3_EXTI11/DCMI_D4/I2S3_ext_SD/SDIO_D3/SPI3_MISO/UART4_RX/USART3_RX/PC11)
- net ENCMOSI1: now also U?.113 (DCMI_D9/I2S3_SD/SDIO_CK/SPI3_MOSI/UART5_TX/USART3_CK/PC12)
- net ENCSCK1: now also U?.111 (DCMI_D8/I2S3_CK/LTDC_R2/SDIO_D2/SPI3_SCK/UART4_TX/USART3_TX/PC10)
- net GNDREF: now also C?.1, D?.1, D?.1, D?.1, D?.1, D?.1, D?.1, D?.1, D?.1, U?.7 (VEE), U?.8 (VSS)
- net SOA1: now also U?.37 (ADC1_IN3/ADC2_IN3/ADC3_IN3/ETH_COL/LTDC_B5/TIM2_CH4/TIM5_CH4/TIM9_CH2/USART2_RX/USB_OTG_HS_ULPI_D0/PA3)
- net SOA2: now also U?.46 (ADC1_IN8/ADC2_IN8/ETH_RXD2/LTDC_R3/TIM1_CH2N/TIM3_CH3/TIM8_CH2N/USB_OTG_HS_ULPI_D1/PB0)
- net SOB1: now also U?.40 (ADC1_IN4/ADC2_IN4/DAC_OUT1/DCMI_HSYNC/I2S3_WS/LTDC_VSYNC/SPI1_NSS/SPI3_NSS/USART2_CK/USB_OTG_HS_SOF/PA4)
- net SOB2: now also U?.47 (ADC1_IN9/ADC2_IN9/ETH_RXD3/LTDC_R6/TIM1_CH3N/TIM3_CH4/TIM8_CH3N/USB_OTG_HS_ULPI_D2/PB1)
- net VDD_3V3: now also C?.2, U?.16 (VDD)
- net VMOT_SENSE: now also U?.13 (PF3/ADC3_IN9/FMC_A3)
- net VSA1: now also U?.42 (ADC1_IN6/ADC2_IN6/DCMI_PIXCK/LTDC_G2/SPI1_MISO/TIM13_CH1/TIM1_BKIN/TIM3_CH1/TIM8_BKIN/PA6)
- net VSA2: now also U?.28 (ADC1_IN12/ADC2_IN12/ADC3_IN12/ETH_TXD2/FMC_SDNE0/I2S2_ext_SD/SPI2_MISO/USB_OTG_HS_ULPI_DIR/PC2)
- net VSB1: now also U?.26 (ADC1_IN10/ADC2_IN10/ADC3_IN10/FMC_SDNWE/USB_OTG_HS_ULPI_STP/PC0)
- net VSB2: now also U?.29 (ADC1_IN13/ADC2_IN13/ADC3_IN13/ETH_TX_CLK/FMC_SDCKE0/I2S2_SD/SPI2_MOSI/USB_OTG_HS_ULPI_NXT/PC3)
- net VSC1: now also U?.27 (ADC1_IN11/ADC2_IN11/ADC3_IN11/ETH_MDC/PC1)
- net VSC2: now also U?.44 (ADC1_IN14/ADC2_IN14/ETH_RXD0/PC4)
- net POT_MUX: now reaches U?.14 (PF4/ADC3_IN14/FMC_A4)
- net POT_MUX: now also U?.3 (X)
- net at R?.2, U?.1: now also R?.1; no longer U?.2 (-) (x2)
- net at R?.1, U?.3 (+): now also D?.3 (x2)
- net at R?.2, U?.7: now also R?.1; no longer U?.6 (-) (x2)
- net at R?.2, U?.8: now also R?.1; no longer U?.9 (-) (x2)
- net at R?.2, U?.14: now also R?.1; no longer U?.13 (-) (x2)
- net at R?.1, U?.5 (+): now also D?.3 (x2)
- net at R?.1, U?.10 (+): now also D?.3 (x2)
- net at R?.1, U?.12 (+): now also D?.3 (x2)
- net POT1: no longer names the net of R?.1, R?.1
- net POT1: now also U?.1 (X4)
- net POT2: no longer names the net of R?.1, R?.1
- net POT2: now also U?.5 (X5)
- net POT3: no longer names the net of R?.1, R?.1
- net POT3: now also U?.2 (X6)
- net POT4: no longer names the net of R?.1, R?.1
- net POT4: now also U?.4 (X7)
- net POT5: no longer names the net of R?.1, R?.1
- net POT5: now also U?.13 (X0)
- net POT6: no longer names the net of R?.1, R?.1
- net POT6: now also U?.14 (X1)
- net POT7: no longer names the net of R?.1, R?.1
- net POT7: now also U?.15 (X2)
- net POT8: no longer names the net of R?.1, R?.1
- net POT8: now also U?.12 (X3)
- net SWO: no longer names the net of P?.8 (SWO)
- new net: R?.2, U?.2 (-) (x2)
- new net: R?.2, U?.6 (-) (x2)
- new net: R?.2, U?.9 (-) (x2)
- new net: R?.2, U?.13 (-) (x2)
- new net POTADDR2: U?.10 (B)
- new net POTADDR3: U?.9 (C)
- new net POTADDRA: U?.11 (A)
- no-connect marks 40 -> 41
Other:
- note added: "ADC1_CH1: \nADC1_CH2: \nADC1_CH3: motor 1 cur A\nADC1_CH4: motor 1 cur B\nADC1_CH5: \nADC1_CH6: motor 1 volt A\nADC1_CH7:\nADC1_CH8:\nADC1_CH9:\nADC1_CH10: motor 1 volt B\nADC1_CH11: motor 1 volt C"
- note added: "ADC2_CH1:\nADC2_CH2:\nADC2_CH3:\nADC2_CH4:\nADC2_CH5:\nADC2_CH6:\nADC2_CH7:\nADC2_CH8: motor 2 cur A\nADC2_CH9: motor 2 cur B\n"
- note added: "TIM1: motor 1\nTIM2: motor 1 enc\nTIM3: motor 1 hall\nTIM4: motor 2 enc\nTIM5: motor 2 hall\nTIM8: motor 2"
- note removed: "Add possibility to bypass"
- note removed: "Investigate up to vcc-2v input range\nConsider TLV2401 or TLV2474 instead\nAdd clipping diodes to output"
- moved on the sheet: C?, D?, L?, P?, R?, U?, U?A, U?B, U?C, U?D

Commit message: change analog out to opamp output
Parts:
- removed D? (x4): BZA408B, symbol SwEmb:BZA408B
- removed P? (x4): CONN_POT_OUT, TerminalBlock_4Ucon:TerminalBlock_4Ucon_1x03_P3.50mm_Horizontal, symbol SwEmb:CONN_POT_OUT
- added C? (x2): CAP_100nF_50V_0402, Capacitor_SMD:C_0402_1005Metric, symbol SwEmb:CAP_100nF_50V_0402
- added P? (x4): CONN_AN_OUT, TerminalBlock_4Ucon:TerminalBlock_4Ucon_1x02_P3.50mm_Horizontal, symbol SwEmb:CONN_AN_OUT
- added P?: CONN_LCD, Connector_PinSocket_2.54mm:PinSocket_2x08_P2.54mm_Vertical, symbol SwEmb:CONN_LCD
- added R? (x4): RES_10K_1%_0402, Resistor_SMD:R_0402_1005Metric, symbol SwEmb:RES_10K_1%_0402
- added R? (x4): RES_5K_1%_0402, Resistor_SMD:R_0402_1005Metric, symbol SwEmb:RES_5K_1%_0402
- added R? (x2): RES_135K_1%_0402, Resistor_SMD:R_0402_1005Metric, symbol SwEmb:RES_135K_1%_0402
- added TP? (x13): Test_Point, TestPoint:TestPoint_Pad_1.0x1.0mm, symbol SwEmb:Test_Point
- added U?: IC_MCP4461, Package_SO:TSSOP-20_4.4x6.5mm_P0.65mm, symbol SwEmb:IC_MCP4461
- added U? (x4): IC_TLV2474, Package_SO:SOIC-14_3.9x8.7mm_P1.27mm, symbol SwEmb:IC_TLV2474
Connections:
- net ECAT_MISO is gone; now on net CANFD_MISO: U?.13 (D1/AD1/EOF/SO/SIO1)
- net ECAT_MOSI is gone; now on net CANFD_MOSI: U?.17 (D0/AD0/WD_STATE/SI/SIO0)
- net ECAT_SCK is gone; now on net CANFD_SCK: U?.19 (D9/AD9/LATCH_IN/SCK)
- net AP_SCL1: now also U?.139 (CAN1_RX/DCMI_D6/ETH_TXD3/I2C1_SCL/LTDC_B6/SDIO_D4/TIM10_CH1/TIM4_CH3/PB8), U?.5 (SCL)
- net AP_SDA1: now also U?.137 (DCMI_VSYNC/FMC_NL/I2C1_SDA/TIM4_CH2/USART1_RX/PB7), U?.6 (SDA)
- net CANFD_CS: now also U?.125 (PG10/DCMI_D2/FMC_NCE4_1/FMC_NE3/LTDC_B2/LTDC_G3)
- net CANFD_INT: now also U?.124 (PG9/DAC_EXTI9/DCMI_VSYNC/FMC_NCE3/FMC_NE2/USART6_RX)
- net CANFD_SOF: now also U?.93 (PG8/ETH_PPS_OUT/FMC_SDCLK/SPI6_NSS/USART6_RTS)
- net CAN_RX1: now also U?.114 (CAN1_RX/FMC_D2/FMC_DA2/PD0)
- net CAN_RX2: now also U?.73 (CAN2_RX/ETH_TXD0/I2C2_SMBA/I2S2_WS/SPI2_NSS/TIM1_BKIN/USART3_CK/USB_OTG_HS_ID/USB_OTG_HS_ULPI_D5/PB12)
- net CAN_STB1: now also U?.89 (PG4/FMC_A14/FMC_BA0)
- net CAN_STB2: now also U?.90 (PG5/FMC_A15/FMC_BA1)
- net CAN_TX1: now also U?.115 (CAN1_TX/FMC_D3/FMC_DA3/PD1)
- net CAN_TX2: now also U?.74 (CAN2_TX/ETH_TXD1/I2S2_CK/SPI2_SCK/TIM1_CH1N/USART3_CTS/USB_OTG_HS_ULPI_D6/USB_OTG_HS_VBUS/PB13)
- net ECAT_CS: now also U?.126 (PG11/ADC1_EXTI11/ADC2_EXTI11/ADC3_EXTI11/DCMI_D3/ETH_TX_EN/FMC_NCE4_2/LTDC_B3)
- net ECAT_IRQ: now also U?.92 (PG7/DCMI_D13/FMC_INT3/LTDC_CLK/USART6_CK)
- net ECAT_RESET: now also U?.91 (PG6/DCMI_D12/FMC_INT2/LTDC_R7)
- net ENCIRQ1: now also U?.68 (PE15/ADC1_EXTI15/ADC2_EXTI15/ADC3_EXTI15/FMC_D12/FMC_DA12/LTDC_R7/TIM1_BKIN)
- net ENCIRQ2: now also U?.42 (ADC1_IN6/ADC2_IN6/DCMI_PIXCK/LTDC_G2/SPI1_MISO/TIM13_CH1/TIM1_BKIN/TIM3_CH1/TIM8_BKIN/PA6)
- net ENCZ2: now also U?.85 (FMC_D0/FMC_DA0/TIM4_CH3/PD14)
- net GNDREF: now also U?.13 (P0B), U?.18 (P2B), U?.3 (P3B), U?.8 (P1B), C?.1, C?.1, P?.2 (GND), P?.2 (GND), P?.2 (GND), P?.2 (GND), R?.2, R?.2, R?.2, R?.2, U?.10 (P1A), U?.11 (V-), U?.11 (V-), U?.11 (V-), U?.11 (V-), U?.13 (P0B), U?.16 (A1), U?.18 (P2B), U?.3 (P3B), U?.7 (GND)
- net OC_ADJ1: now also U?.15 (PF5/ADC3_IN15/FMC_A5), R?.1, U?.19 (P2W)
- net POT_MUX: now also TP?.1
- net VDD_3V3: now also C?.2, R?.2, U?.1 (P3A), U?.10 (P1A), U?.11 (P0A), U?.17 (VDD), U?.20 (P2A), C?.2, R?.2, R?.2, U?.17 (VDD), U?.4 (HVC/A0)
- net VDD_5V: now also C?.2, U?.4 (V+), U?.4 (V+), U?.4 (V+), U?.4 (V+); no longer C?.2, R?.2, U?.17 (VDD)
- net VSA1: now also U?.45 (ADC1_IN15/ADC2_IN15/ETH_RXD1/PC5); no longer U?.42 (ADC1_IN6/ADC2_IN6/DCMI_PIXCK/LTDC_G2/SPI1_MISO/TIM13_CH1/TIM1_BKIN/TIM3_CH1/TIM8_BKIN/PA6)
- net OC_ADJ2: now reaches U?.18 (PF6/ADC3_IN4/FMC_NIORD/SAI1_SD_B/SPI5_NSS/TIM10_CH1/UART7_RX)
- net OC_ADJ2: now also R?.1, U?.2 (P3W)
- net at R?.1, R?.1, U?.1 (X4): now also TP?.1
- net at R?.1, R?.1, U?.5 (X5): now also TP?.1
- net at R?.1, R?.1, U?.2 (X6): now also TP?.1
- net at R?.1, R?.1, U?.4 (X7): now also TP?.1
- net at R?.1, R?.1, U?.13 (X0): now also TP?.1
- net at R?.1, R?.1, U?.14 (X1): now also TP?.1
- net at R?.1, R?.1, U?.15 (X2): now also TP?.1
- net at R?.1, R?.1, U?.12 (X3): now also TP?.1
- net at U?.12 (P0W): now also TP?.1, U?.10 (+)
- net at U?.19 (P2W): now also TP?.1, U?.5 (+)
- net at U?.2 (P3W): now also TP?.1, U?.3 (+)
- net at U?.9 (P1W): now also TP?.1, U?.12 (+)
- net ENCAF1: no longer names the net of U?.2 (~AFAULT)
- net ENCAF2: no longer names the net of U?.2 (~AFAULT)
- net ENCBF1: no longer names the net of U?.21 (~BFAULT)
- net ENCBF2: no longer names the net of U?.21 (~BFAULT)
- net ENCSGCTRL1: no longer names the net of U?.14 (DI/TTL2)
- net ENCSGCTRL2: no longer names the net of U?.14 (DI/TTL2)
- net ENCSHCTRL1: no longer names the net of U?.30 (DI/TTL3)
- net ENCSHCTRL2: no longer names the net of U?.30 (DI/TTL3)
- net ENCSYCTRL1: no longer names the net of U?.18 (DI/TTLY)
- net ENCSYCTRL2: no longer names the net of U?.18 (DI/TTLY)
- net ENCSYF1: no longer names the net of U?.19 (~YFAULT)
- net ENCSYF2: no longer names the net of U?.19 (~YFAULT)
- net ENCZF1: no longer names the net of U?.20 (~ZFAULT)
- net ENCZF2: no longer names the net of U?.20 (~ZFAULT)
- new net: P?.1 (AN), R?.1, U?.1
- new net: R?.1, R?.2, U?.2 (-)
- new net: R?.1, R?.2, U?.6 (-)
- new net: P?.1 (AN), R?.1, U?.7
- new net: P?.1 (AN), R?.1, U?.8
- new net: R?.1, R?.2, U?.9 (-)
- new net: R?.1, R?.2, U?.13 (-)
- new net: P?.1 (AN), R?.1, U?.14
- new net MOCP_RESET: U?.15 (~RESET)
- new net MOCP_WP: U?.14 (~WP)
- no-connect marks 41 -> 57
Other:
- note added: "Add opamps to voltage sensing"
- note added: "Encoder Interface Power SW"
- note added: "Implement industrial digital inputs with 30v tolerance"
- note added: "Overcurrent limit ADJ"
- note added: "Wide input range: -40V to +40V"
- note removed: "Add possibility to bypass power"
- moved on the sheet: C?, U?
