File: motordriver-2x.sch (KiCad schematic (older format))
At the start: 525 parts, among them J1 USB_B_Micro, J2 CONN_RJ45_MAG, J3 CONN_RJ45_MAG, P1 CONN_SWITCH, P10 CONN_SENSOR, P11 CONN_SENSOR, P12 CONN_SENSOR, P13 CONN_SENSOR, P14 CONN_SENSOR, P15 CONN_SENSOR, P16 CONN_SENSOR, P17 CONN_DEBUG_2R, P18 CONN_POWER_41A, P19 CONN_CAN, P2 CONN_SWITCH, P20 CONN_CAN, P21 CONN_AN_OUT, P22 CONN_AN_OUT, P23 CONN_POWER_10A, P24 CONN_CAN, P25 CONN_LCD, P26 CONN_AN_OUT, P27 CONN_AN_OUT, P28 CONN_UEXT, P29 CONN_LED, P3 CONN_SWITCH, P30 CONN_LED, P31 CONN_LED, P32 CONN_LED, P33 CONN_LED, P34 CONN_LED, P35 CONN_LED, P36 CONN_LED, P37 CONN_ENCODER, P38 CONN_SENSOR, P39 CONN_SENSOR, P4 CONN_SWITCH, P40 CONN_SENSOR, P41 CONN_ENCODER, P42 CONN_SENSOR, P43 CONN_SENSOR, P44 CONN_SENSOR, P45 CONN_MOTOR, P46 CONN_MOTOR, P47 CONN_HALL, P48 CONN_HALL, P5 CONN_SWITCH, P6 CONN_SWITCH, P7 CONN_SWITCH, P8 CONN_SWITCH, P9 CONN_SENSOR, Q1 Q_NMOS_2X_100V_70A, Q2 Q_NMOS_2X_100V_70A, Q3 Q_NMOS_2X_100V_70A, Q4 Q_NMOS_2X_100V_70A, Q5 Q_NMOS_2X_100V_70A, Q6 Q_NMOS_2X_100V_70A, U1 IC_MIC2026, U10 IC_MCP4461, U11 IC_MCP2517FD-xJHA, U12 IC_STM32F429ZET6, U13 IC_MCP23S17, U14 IC_TPS54360DDA, U15 IC_TJA1044GT3, U16 IC_TLV2474, U17 IC_M24C16, U18 IC_USBLC6-2, U19 IC_TPS62147RGXR, U2 IC_MAX6818, U20 IC_TLV5533, U21 IC_LP55231, U22 IC_TLV5533, U23 IC_MAX14890, U24 IC_MAX14890, U25 IC_MIC2026, U26 IC_TLV2474, U27 IC_USBLC6-2, U28 IC_USBLC6-2, U29 IC_MCP4461, U3 IC_TLV2474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

Commit message: draft sent
Connections:
- wire segments 1765 -> 1774
Other:
- note added: "- Capable of driving two PMSM or DC motors @ 48V, 20A\n- Automatic overcurrent protection with adjustable current limit\n- Break resistor support\n- Versatile encoder interface supporting SE, RS-422 and DHTL encoders\n- 3 extra +-40 inputs per motor for high voltage industrial sensors\n- Motor hall sensor support\n- Amplified back emf feedback for better sensorless control\n- 2x CAN2.0B\n- CANFD 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"
- note added: "ADC1"
- note added: "ADC2"
- note added: "Quick Design Summary"
- note added: "STM32 Peripheral Assignments"
- note added: "This is a draft\nIncomplete!"
- note added: "Timers"
- moved on the sheet: C100, C101, C102, C103, C104, C105, C106, C107, C108, C109, C110, C111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

Commit message: start reviewing the schematic
Parts:
- added C?: CAP_100nF_100V_0603, Capacitor_SMD:C_0603_1608Metric, symbol SwEmb:CAP_100nF_50V_0402
- C102, C111, C114, C117, C118, C119, C86, C93, C95, C96, C99: symbol SwEmb:CAP_100nF_100V_0603 -> SwEmb:CAP_100nF_50V_0402
- gave numbers to parts that had none: 11
Connections:
- wire segments 1774 -> 1770
Other:
- moved on the sheet: C103, C104, C112, C113, C114, C118

Commit message: review start
Parts:
- added C152, C153, C154, C155, C156, C157: CAP_100nF_50V_0402, Capacitor_SMD:C_0402_1005Metric, symbol SwEmb:CAP_100nF_50V_0402
- added D31: LED_RED_0603, LED_SMD:LED_0603_1608Metric, symbol SwEmb:LED_RED_0603
- added P50, P51: CONN_SENSOR, TerminalBlock_4Ucon:TerminalBlock_4Ucon_1x03_P3.50mm_Horizontal, symbol SwEmb:CONN_SENSOR
- added R198: RES_470R_1%_0402, Resistor_SMD:R_0402_1005Metric, symbol SwEmb:RES_470R_1%_0402
- added R199, R201: RES_10K_1%_0402, Resistor_SMD:R_0402_1005Metric, symbol SwEmb:RES_10K_1%_0402
- added R200, R202: RES_NTC_10K_402, Resistor_SMD:R_0402_1005Metric, symbol SwEmb:RES_NTC_10K_402
- added U36: IC_TXS0108, Package_SO:TSSOP-20_4.4x6.5mm_P0.65mm, symbol SwEmb:IC_TXS0108
- C102, C111, C114, C117, C118, C119, C86, C93, C95, C96, C99: value CAP_100nF_100V_0603 -> CAP_100nF_50V_0402; footprint Capacitor_SMD:C_0603_1608Metric -> Capacitor_SMD:C_0402_1005Metric; Availability 121849 In Stock -> 120297 In Stock; Description Multilayer Ceramic Capacitors MLCC - SMD/SMT 100K pF 10% 10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 -> Multilayer Ceramic Capacitors MLCC - SMD/SMT 100K pF 50Volt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; MPN CC0603KRX7R0BB104 -> CC0402KRX5R9BB104; Price 0.183 EUR -> 0.087 EUR
- C151: renamed from C?; value CAP_100nF_100V_0603 -> CAP_100nF_50V_0402; footprint Capacitor_SMD:C_0603_1608Metric -> Capacitor_SMD:C_0402_1005Metric; Availability 121849 In Stock -> 120297 In Stock; Description Multilayer Ceramic Capacitors MLCC - SMD/SMT 100K pF 10% 10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 -> Multilayer Ceramic Capacitors MLCC - SMD/SMT 100K pF 50Volt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; MPN CC0603KRX7R0BB104 -> CC0402KRX5R9BB104; Price 0.183 EUR -> 0.087 EUR
Connections:
- net labels added: PWM_IN1, PWM_IN2, TEMP_MOT1, TEMP_MOT2
- wire segments 1770 -> 1802
Other:
- note added: "PWM/PPM IN"

Commit message: continue schematic review: capacitors
Parts:
- removed C32: CAP_100nF_50V_0402, Capacitor_SMD:C_0402_1005Metric, symbol SwEmb:CAP_100nF_50V_0402
- removed C51: CAP_2.2uF_16V_0402, Capacitor_SMD:C_0402_1005Metric, symbol SwEmb:CAP_2.2uF_16V_0402
- C13: value CAP_100nF_50V_0402 -> CAP_2.2uF_16V_0402; symbol SwEmb:CAP_100nF_50V_0402 -> SwEmb:CAP_2.2uF_16V_0402; Availability 120297 In Stock -> 113017 In Stock; Description Multilayer Ceramic Capacitors MLCC - SMD/SMT 100K pF 50Volt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 -> Multilayer Ceramic Capacitors MLCC - SMD/SMT 0402 16Vdc 2.2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; MPN CC0402KRX5R9BB104 -> GRT155C81C225KE13D; Price 0.087 EUR -> 0.271 EUR
- C141, C142: value CAP_2.2nF_50V_0603 -> CAP_22nF_50V_0402; footprint Capacitor_SMD:C_0603_1608Metric -> Capacitor_SMD:C_0402_1005Metric; symbol SwEmb:CAP_2.2nF_50V_0603 -> SwEmb:CAP_22nF_50V_0402; Availability 116641 In Stock -> 76047 In Stock; Description Multilayer Ceramic Capacitors MLCC - SMD/SMT CGA 0603 50V 0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 -> Multilayer Ceramic Capacitors MLCC - SMD/SMT 0402 0.022uF 5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; MPN CGA3E2X7R1H223K080AA -> GCM155R71H223JA55D
- C147, C148: value CAP_2.2uF_100V_1210 -> CAP_2.2uF_16V_0402; footprint Capacitor_SMD:C_1210_3225Metric -> Capacitor_SMD:C_0402_1005Metric; symbol SwEmb:CAP_2.2uF_100V_1210 -> SwEmb:CAP_2.2uF_16V_0402; Availability 12161 In Stock -> 113017 In Stock; Description Multilayer Ceramic Capacitors MLCC - SMD/SMT 2.2uF 100V X7R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 -> Multilayer Ceramic Capacitors MLCC - SMD/SMT 0402 16Vdc 2.2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; MPN HMJ325AB7225KMHT -> GRT155C81C225KE13D; Price 1.00 EUR -> 0.271 EUR
- C45: value CAP_10uF_35V_0603 -> CAP_10uF_25V_0805; footprint Capacitor_SMD:C_0603_1608Metric -> Capacitor_SMD:C_0805_2012Metric; symbol SwEmb:CAP_10uF_35V_0603 -> SwEmb:CAP_10uF_25V_0805; Availability 1829 In Stock -> 196753 In Stock; Description Multilayer Ceramic Capacitors MLCC - SMD/SMT 0603 10uF 35vo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 -> Multilayer Ceramic Capacitors MLCC - SMD/SMT 0805 10uF 25vo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; MPN GRM188R6YA106MA73D -> GRM21BR61E106MA73L; Price 0.437 EUR -> 0.262 EUR
- C49: symbol SwEmb:CAP_100nF_50V_0402 -> SwEmb:CAP_10uF_25V_0805
- R200, R202: Availability (none) -> 199483 In Stock; Description (none) -> NTC (Negative Temperature Coefficient) Thermistors THERMIST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; LifeCycle (none) -> OK; Price (none) -> 0.087 EUR; Vendor (none) -> Mouser
- U36: Availability 48961 In Stock -> 43158 In Stock
- Y2: Availability 5608 In Stock -> 4328 In Stock
Connections:
- wire segments 1802 -> 1793
Other:
- moved on the sheet: C120, C31, C37, C49

Commit message: review diodes
Parts:
- removed D15: D_MM3Z3V3B, Diode_SMD:D_SOD-323F, symbol SwEmb:D_MM3Z3V3B
- removed D30: D_BAT54, Diode_SMD:D_SOD-123, symbol SwEmb:D_BAT54
- removed U20: IC_TLV5533, Package_TO_SOT_SMD:SOT-23-5, symbol SwEmb:IC_TLV5533
- added C32: CAP_100nF_50V_0402, Capacitor_SMD:C_0402_1005Metric, symbol SwEmb:CAP_100nF_50V_0402
- added D32: D_BAT54, Diode_SMD:D_SOD-123, symbol SwEmb:D_BAT54
- added F1: FUSE_3A_9750, CUSTOM:Fuse_Littlefuse_9750, symbol SwEmb:FUSE_3A_9750
- added R203, R204, R205, R206, R207, R208: RES_10K_1%_0402, Resistor_SMD:R_0402_1005Metric, symbol SwEmb:RES_10K_1%_0402
- added U20: IC_TLV75533, Package_TO_SOT_SMD:SOT-23-5, symbol SwEmb:IC_TLV75533
- added unit 2 of U26
- added unit 3 of U26
- added unit 4 of U26
- C49: value CAP_100nF_50V_0402 -> CAP_10uF_25V_0805; footprint Capacitor_SMD:C_0402_1005Metric -> Capacitor_SMD:C_0805_2012Metric; Availability 120297 In Stock -> 196753 In Stock; Description Multilayer Ceramic Capacitors MLCC - SMD/SMT 100K pF 50Volt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 -> Multilayer Ceramic Capacitors MLCC - SMD/SMT 0805 10uF 25vo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; MPN CC0402KRX5R9BB104 -> GRM21BR61E106MA73L; Price 0.087 EUR -> 0.262 EUR
- C63, C82, C83: value CAP_100nF_100V_0603 -> CAP_100nF_50V_0402; footprint Capacitor_SMD:C_0603_1608Metric -> Capacitor_SMD:C_0402_1005Metric; symbol SwEmb:CAP_100nF_100V_0603 -> SwEmb:CAP_100nF_50V_0402; Availability 121849 In Stock -> 120297 In Stock; Description Multilayer Ceramic Capacitors MLCC - SMD/SMT 100K pF 10% 10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 -> Multilayer Ceramic Capacitors MLCC - SMD/SMT 100K pF 50Volt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; MPN CC0603KRX7R0BB104 -> CC0402KRX5R9BB104; Price 0.183 EUR -> 0.087 EUR
- C87, C88, C91, C92: value CAP_1uF_10V_0402 -> CAP_2.2uF_16V_0402; symbol SwEmb:CAP_1uF_10V_0402 -> SwEmb:CAP_2.2uF_16V_0402; Availability 19231817 In Stock -> 113017 In Stock; Description Multilayer Ceramic Capacitors MLCC - SMD/SMT 1uF 10V X5R 10% -> Multilayer Ceramic Capacitors MLCC - SMD/SMT 0402 16Vdc 2.2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; MPN CC0402KRX5R6BB105 -> GRT155C81C225KE13D; Price 0.148 EUR -> 0.271 EUR
- D10, D11, D13: value D_ESDCAN06 -> D_ESDCAN03; symbol SwEmb:D_ESDCAN06 -> SwEmb:D_ESDCAN03; MPN ESDCAN06-2BWY -> ESDCAN03-2BWY
- D16: value D_MM3Z3V3B -> D_SZ1SMB5913BT3G; footprint Diode_SMD:D_SOD-323F -> Diode_SMD:D_SMB; symbol SwEmb:D_MM3Z3V3B -> SwEmb:D_SZ1SMB5913BT3G; MPN MM3Z3V3B -> SZ1SMB5913BT3G
- R196, R197: symbol SwEmb:RES_135K_1%_0402 -> SwEmb:RES_10K_1%_0402
- U22: value IC_TLV5533 -> IC_TLV75533; symbol SwEmb:IC_TLV5533 -> SwEmb:IC_TLV75533
- renumbered U26 to U33, U33 to U35, U26 to U35
Connections:
- wire segments 1793 -> 1836
Other:
- note added: "Unused sections wiring"
- moved on the sheet: C54, P23, P28, R197

Commit message: schematic review
Parts:
- D16: Availability 110855 In Stock -> 2800 In Stock; Description Zener Diodes Diode Zener 3.3V 200mW 2% -> Zener Diodes ZEN SMB REG 3W; Price 0.183 EUR -> 0.55 EUR
- J1: footprint Connector_USB:USB_Micro-B_GCT_USB3076-30-A -> CUSTOM:USB_Micro-B_GCT_USB3076-30-A
- J2, J3: MPN (none) -> 7499010121A
- R196, R197: value RES_135K_1%_0402 -> RES_10K_1%_0402; Availability 147765 In Stock -> 1813839 In Stock; Description Thick Film Resistors - SMD 135 kOhms 1% -> Thick Film Resistors - SMD 1/16watt 10Kohms 1% Commercial U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; LifeCycle OK -> New Product; MPN RC0402FR-135K1L -> CRCW040210K0FKEDC; Price 0.087 EUR -> 0.114 EUR
Changed lines of the file:
@@
 F 3 "" H 22550 18925 50  0001 C CNN
 F 4 "7499010121A" H -4400 3200 50  0001 C CNN "MFN"
+F 5 "7499010121A" H 0   0   50  0001 C CNN "MPN"
 	1    22450 18325
 	1    0    0    -1
@@
 U 1 1 79833276
 P 19100 18925
-F 0 "R110" V 19050 18800 50  0000 C CNN
+F 0 "R110" V 19050 18750 50  0000 C CNN
 F 1 "RES_10K_1%_0402" H 19130 18885 50  0001 L CNN
 F 2 "Resistor_SMD:R_0402_1005Metric" H 19030 18845 50  0001 C CNN
@@
 U 1 1 79834610
 P 19000 18925
-F 0 "R108" V 18950 18800 50  0000 C CNN
+F 0 "R108" V 18950 18750 50  0000 C CNN
 F 1 "RES_10K_1%_0402" H 19030 18885 50  0001 L CNN
 F 2 "Resistor_SMD:R_0402_1005Metric" H 18930 18845 50  0001 C CNN
@@
 U 1 1 7A2111E1
 P 19200 18925
-F 0 "R113" V 19150 18800 50  0000 C CNN
+F 0 "R113" V 19150 18750 50  0000 C CNN
 F 1 "RES_10K_1%_0402" H 19230 18885 50  0001 L CNN
 F 2 "Resistor_SMD:R_0402_1005Metric" H 19130 18845 50  0001 C CNN
@@
 U 1 1 7AC16226
 P 19300 18925
-F 0 "R116" V 19250 18800 50  0000 C CNN
+F 0 "R116" V 19250 18750 50  0000 C CNN
 F 1 "RES_10K_1%_0402" H 19330 18885 50  0001 L CNN
 F 2 "Resistor_SMD:R_0402_1005Metric" H 19230 18845 50  0001 C CNN
@@
 F 3 "" H 22550 17575 50  0001 C CNN
 F 4 "7499010121A" H -4400 3200 50  0001 C CNN "MFN"
+F 5 "7499010121A" H 0   0   50  0001 C CNN "MPN"
 	1    22450 16975
 	1    0    0    -1
@@
 F 1 "D_SZ1SMB5913BT3G" H 13725 21610 50  0001 C CNN
 F 2 "Diode_SMD:D_SMB" H 13625 21690 50  0001 C CNN
-F 3 "https://www.mouser.com/datasheet/2/308/MM3Z10VB-1301283.pdf" H 13725 21790 50  0001 C CNN
+F 3 "https://www.mouser.com/datasheet/2/308/1SMB5913BT3-D-1292981.pdf" H 13725 21790 50  0001 C CNN
 F 4 "SZ1SMB5913BT3G" H 13725 21700 39  0001 C CNN "MPN"
-F 5 "110855 In Stock" H 0   0   50  0001 C CNN "Availability"
-F 6 "Zener Diodes Diode Zener 3.3V 200mW 2%" H 0   0   50  0001 C CNN "Description"
+F 5 "2800 In Stock" H 0   0   50  0001 C CNN "Availability"
+F 6 "Zener Diodes ZEN SMB REG 3W" H 0   0   50  0001 C CNN "Description"
 F 7 "OK" H 0   0   50  0001 C CNN "LifeCycle"
-F 8 "0.183  EUR" H 0   0   50  0001 C CNN "Price"
+F 8 "0.55  EUR" H 0   0   50  0001 C CNN "Price"
 F 9 "Mouser" H 0   0   50  0001 C CNN "Vendor"
 	1    13725 21700
@@
 F 0 "J1" H 8805 11067 50  0000 C CNN
 F 1 "USB_B_Micro" H 8805 10976 50  0000 C CNN
-F 2 "Connector_USB:USB_Micro-B_GCT_USB3076-30-A" H 8900 10550 50  0001 C CNN
+F 2 "CUSTOM:USB_Micro-B_GCT_USB3076-30-A" H 8900 10550 50  0001 C CNN
 F 3 "https://www.mouser.com/datasheet/2/18/10118193-1361773.pdf" H 8750 10600 50  0001 C CNN
 F 4 "10118193-0001LF" H 8900 11150 50  0001 C CNN "MPN"
@@
 P 7475 20225
 F 0 "R197" H 7534 20225 50  0000 L CNN
-F 1 "RES_135K_1%_0402" H 7505 20185 50  0001 L CNN
+F 1 "RES_10K_1%_0402" H 7505 20185 50  0001 L CNN
 F 2 "Resistor_SMD:R_0402_1005Metric" H 7405 20145 50  0001 C CNN
-F 3 "https://www.mouser.com/datasheet/2/447/yageo_01152019_DESIGN_KITS_8_2012-1522572.pdf" H 7505 20245 50  0001 C CNN
-F 4 "RC0402FR-135K1L" H 7605 20345 50  0001 C CNN "MPN"
-F 5 "147765 In Stock" H 7475 20225 50  0001 C CNN "Availability"
-F 6 "Thick Film Resistors - SMD 135 kOhms 1%" H 7475 20225 50  0001 C CNN "Description"
-F 7 "OK" H 7475 20225 50  0001 C CNN "LifeCycle"
-F 8 "0.087  EUR" H 7475 20225 50  0001 C CNN "Price"
+F 3 "" H 7505 20245 50  0001 C CNN
+F 4 "CRCW040210K0FKEDC" H 7605 20345 50  0001 C CNN "MPN"
+F 5 "1813839 In Stock" H 7475 20225 50  0001 C CNN "Availability"
+F 6 "Thick Film Resistors - SMD 1/16watt 10Kohms 1% Commercial Use" H 7475 20225 50  0001 C CNN "Description"
+F 7 "New Product" H 7475 20225 50  0001 C CNN "LifeCycle"
+F 8 "0.114  EUR" H 7475 20225 50  0001 C CNN "Price"
 F 9 "Mouser" H 7475 20225 50  0001 C CNN "Vendor"
 	1    7475 20225
@@
 P 7275 19875
 F 0 "R196" V 7171 19875 50  0000 C CNN
-F 1 "RES_135K_1%_0402" H 7305 19835 50  0001 L CNN
+F 1 "RES_10K_1%_0402" H 7305 19835 50  0001 L CNN
 F 2 "Resistor_SMD:R_0402_1005Metric" H 7205 19795 50  0001 C CNN
-F 3 "https://www.mouser.com/datasheet/2/447/yageo_01152019_DESIGN_KITS_8_2012-1522572.pdf" H 7305 19895 50  0001 C CNN
-F 4 "RC0402FR-135K1L" H 7405 19995 50  0001 C CNN "MPN"
-F 5 "147765 In Stock" H 7275 19875 50  0001 C CNN "Availability"
-F 6 "Thick Film Resistors - SMD 135 kOhms 1%" H 7275 19875 50  0001 C CNN "Description"
-F 7 "OK" H 7275 19875 50  0001 C CNN "LifeCycle"
-F 8 "0.087  EUR" H 7275 19875 50  0001 C CNN "Price"
+F 3 "" H 7305 19895 50  0001 C CNN
+F 4 "CRCW040210K0FKEDC" H 7405 19995 50  0001 C CNN "MPN"
+F 5 "1813839 In Stock" H 7275 19875 50  0001 C CNN "Availability"
+F 6 "Thick Film Resistors - SMD 1/16watt 10Kohms 1% Commercial Use" H 7275 19875 50  0001 C CNN "Description"
+F 7 "New Product" H 7275 19875 50  0001 C CNN "LifeCycle"
+F 8 "0.114  EUR" H 7275 19875 50  0001 C CNN "Price"
 F 9 "Mouser" H 7275 19875 50  0001 C CNN "Vendor"
 	1    7275 19875

Commit message: review footprints for switches and sensors
Parts:
- J2, J3: footprint Connector_RJ:RJ45_Tranformer -> CUSTOM:RJ45_Tranformer; Availability (none) -> 202 In Stock; Description (none) -> Modular Connectors / Ethernet Connectors WE-RJ45 Intgtd XFM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; LifeCycle (none) -> OK; Price (none) -> 5.72 EUR; Vendor (none) -> Mouser
- P1, P2, P3, P4, P5, P6, P7, P8: footprint TerminalBlock_4Ucon:TerminalBlock_4Ucon_1x02_P3.50mm_Horizontal -> CUSTOM:TerminalBlock_4Ucon_1x02_P3.50mm_Horizontal; Availability 2043 In Stock -> 1435 In Stock; Description Pluggable Terminal Blocks WR-TBL PCB Model3211 2Pin 3.5mm V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 -> Pluggable Terminal Blocks WR-TBL PCB Model3221 2Pin 3.5mm H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; MPN 691321100002 -> 691322110002
- P10, P11, P12, P13, P14, P15, P16, P38, P39, P40, P42, P43, P44, P50, P51, P9: footprint TerminalBlock_4Ucon:TerminalBlock_4Ucon_1x03_P3.50mm_Horizontal -> CUSTOM:TerminalBlock_4Ucon_1x03_P3.50mm_Horizontal; MPN 691321100003 -> 691322110003

Commit message: component level review almost done on connectors
Add a bunch of modified footprints and push latest schematic
Parts:
- P1, P2, P3, P4, P5, P6, P7, P8: footprint CUSTOM:TerminalBlock_4Ucon_1x02_P3.50mm_Horizontal -> CUSTOM:CONN_SWITCH
- P10, P11, P12, P13, P14, P15, P16, P38, P39, P40, P42, P43, P44, P50, P51, P9: footprint CUSTOM:TerminalBlock_4Ucon_1x03_P3.50mm_Horizontal -> CUSTOM:CONN_SENSOR
- P17: footprint Connector_PinSocket_2.54mm:PinSocket_2x05_P2.54mm_Vertical -> Connector_IDC:IDC-Header_2x05_P2.54mm_Vertical
- P19, P20, P24: footprint TerminalBlock_4Ucon:TerminalBlock_4Ucon_1x03_P3.50mm_Horizontal -> CUSTOM:CONN_CAN; MPN 691321100003 -> 691322110003
- P21, P22, P26, P27: footprint TerminalBlock_4Ucon:TerminalBlock_4Ucon_1x02_P3.50mm_Horizontal -> CUSTOM:CONN_AN_OUT; MPN 691321100002 -> 691322110002
- P23: footprint TerminalBlock_4Ucon:TerminalBlock_4Ucon_1x02_P3.50mm_Horizontal -> CUSTOM:CONN_POWER_10A; MPN 691321100002 -> 691322110002
- P25: footprint Connector_PinSocket_2.54mm:PinSocket_2x08_P2.54mm_Vertical -> CUSTOM:CONN_LCD
- P28: footprint Connector_PinSocket_2.54mm:PinSocket_2x05_P2.54mm_Vertical -> CUSTOM:CONN_UEXT
- P29, P30, P31, P32, P33, P34, P35, P36: footprint TerminalBlock_4Ucon:TerminalBlock_4Ucon_1x02_P3.50mm_Horizontal -> CUSTOM:CONN_LED; MPN 691321100002 -> 691322110002
- P47, P48: footprint TerminalBlock_MetzConnect:TerminalBlock_MetzConnect_Type059_RT06305HBWC_1x05_P3.50mm_Horizontal -> CUSTOM:CONN_HALL
- P49: footprint TerminalBlock_4Ucon:TerminalBlock_4Ucon_1x02_P3.50mm_Horizontal -> CUSTOM:CONN_BRKRES; MPN 691321100002 -> 691322110002
