File: motordriver-2x.kicad_pcb (KiCad board)
At the start: 2 copper layers, 514 parts, among them J1 USB_B_Micro, J2 CONN_RJ45_MAG, J3 CONN_RJ45_MAG, P1 CONN_SWITCH, P10 CONN_SENSOR, P11 CONN_SENSOR, P12 CONN_SENSOR, P13 CONN_SENSOR, P14 CONN_SENSOR, P15 CONN_SENSOR, P16 CONN_SENSOR, P17 CONN_DEBUG_2R, P18 CONN_POWER_41A, P19 CONN_CAN, P2 CONN_SWITCH, P20 CONN_CAN, P21 CONN_AN_OUT, P22 CONN_AN_OUT, P23 CONN_POWER_10A, P24 CONN_CAN, P25 CONN_LCD, P26 CONN_AN_OUT, P27 CONN_AN_OUT, P28 CONN_UEXT, P29 CONN_LED, P3 CONN_SWITCH, P30 CONN_LED, P31 CONN_LED, P32 CONN_LED, P33 CONN_LED, P34 CONN_LED, P35 CONN_LED, P36 CONN_LED, P37 CONN_ENCODER, P38 CONN_SENSOR, P39 CONN_SENSOR, P4 CONN_SWITCH, P40 CONN_SENSOR, P41 CONN_ENCODER, P42 CONN_SENSOR, P43 CONN_SENSOR, P44 CONN_SENSOR, P45 CONN_MOTOR, P46 CONN_MOTOR, P47 CONN_HALL, P48 CONN_HALL, P5 CONN_SWITCH, P6 CONN_SWITCH, P7 CONN_SWITCH, P8 CONN_SWITCH, P9 CONN_SENSOR, Q1 Q_NMOS_2X_100V_70A, Q2 Q_NMOS_2X_100V_70A, Q3 Q_NMOS_2X_100V_70A, Q4 Q_NMOS_2X_100V_70A, Q5 Q_NMOS_2X_100V_70A, Q6 Q_NMOS_2X_100V_70A, U1 IC_MIC2026, U10 IC_MCP4461, U11 IC_MCP2517FD-xJHA, U12 IC_STM32F429ZET6, U13 IC_MCP23S17, U14 IC_TPS54360DDA, U15 IC_TJA1044GT3, U16 IC_TLV2474, U17 IC_M24C16, U18 IC_USBLC6-2, U19 IC_TPS62147RGXR, U2 IC_MAX6818, U20 IC_TLV5533, U21 IC_LP55231, U22 IC_TLV5533, U23 IC_MAX14890, U24 IC_MAX14890, U25 IC_MIC2026, U26 IC_TLV2474, U27 IC_USBLC6-2, U28 IC_USBLC6-2, U29 IC_MCP4461, U3 IC_TLV2474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

Commit message: fix footprints
Parts:
- C84, C85: value CAP_2.2uF_100V_1210 -> CAP_2.2uF_16V_0402; footprint Capacitor_SMD:C_1210_3225Metric -> Capacitor_SMD:C_0402_1005Metric
- moved U31 251.8 mm to (175.7, -56.8)
- moved R157 202.3 mm to (221.6, -31.4)
- moved C89 191.2 mm to (169.0, -56.6)
- moved C145 190.3 mm to (232.0, -20.0)
- moved R103 178.6 mm to (221.5, -53.4), turned to 180 degrees
- moved Q5 177.4 mm to (226.8, -46.6), turned to 270 degrees
- moved R171 176.2 mm to (221.6, -43.6), turned to 180 degrees
- moved R170 175.9 mm to (221.6, -49.6), turned to 180 degrees
- moved R140 174.5 mm to (207.0, -39.0)
- moved R114 174.5 mm to (189.0, -35.0)
- moved R169 172.0 mm to (221.6, -48.4), turned to 180 degrees
- moved C105 165.1 mm to (185.0, -12.0)
- moved R102 165.0 mm to (198.0, -22.0)
- moved R156 163.9 mm to (221.6, -32.6)
- moved R117 163.5 mm to (199.0, -34.0)
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
Commit message: start reviewing the schematic
Parts:
- added D27: D_BAT54, Diode_SMD:D_SOD-123, F.Cu at (202.9, 147.0)
- added D28: D_CDBC5100, Diode_SMD:D_SMC, F.Cu at (179.9, 160.5)
- added D29: D_STPS41H100, Package_TO_SOT_SMD:TO-263-2, F.Cu at (183.3, 151.5)
- added D30: D_BAT54, Diode_SMD:D_SOD-123, F.Cu at (187.2, 158.3)
- added P49: CONN_BRKRES, TerminalBlock_4Ucon:TerminalBlock_4Ucon_1x02_P3.50mm_Horizontal, F.Cu at (194.3, 157.0)
- added Q7: Q_PNP_BC856, Package_TO_SOT_SMD:SOT-23, F.Cu at (186.6, 161.3)
- added Q8: Q_NMOS_BUK9875, Package_TO_SOT_SMD:SOT-223, F.Cu at (196.1, 149.4)
- added R195: RES_10K_1%_0402, Resistor_SMD:R_0402_1005Metric, F.Cu at (206.1, 146.3)
- added R196: RES_135K_1%_0402, Resistor_SMD:R_0402_1005Metric, F.Cu at (185.7, 163.6)
- added R197: RES_135K_1%_0402, Resistor_SMD:R_0402_1005Metric, F.Cu at (189.1, 160.0)
- added TP41: Test_Point, TestPoint:TestPoint_Pad_1.0x1.0mm, F.Cu at (189.3, 162.1)
Connections:
- C15 pad 1: VMOT -> Net-(C15-Pad1)
- D9 pad 1: VMOT -> BREAK
- P18 pad 1: VMOT -> BREAK
- R39 pad 2: VMOT -> Net-(C15-Pad1)
- TP10 pad 1: VMOT -> Net-(C15-Pad1)

Commit message: review start
Parts:
- added C151: CAP_100nF_100V_0603, Capacitor_SMD:C_0603_1608Metric, F.Cu at (243.2, 111.4)
- added C152: CAP_100nF_50V_0402, Capacitor_SMD:C_0402_1005Metric, F.Cu at (244.3, 112.7)
- added C153: CAP_100nF_50V_0402, Capacitor_SMD:C_0402_1005Metric, F.Cu at (241.3, 113.7)
- added C154: CAP_100nF_50V_0402, Capacitor_SMD:C_0402_1005Metric, F.Cu at (239.6, 114.8)
- added C155: CAP_100nF_50V_0402, Capacitor_SMD:C_0402_1005Metric, F.Cu at (239.6, 113.8)
- added C156: CAP_100nF_50V_0402, Capacitor_SMD:C_0402_1005Metric, F.Cu at (241.3, 114.7)
- added C157: CAP_100nF_50V_0402, Capacitor_SMD:C_0402_1005Metric, F.Cu at (239.6, 115.8)
- added D31: LED_RED_0603, LED_SMD:LED_0603_1608Metric, F.Cu at (240.3, 111.5)
- added P50: CONN_SENSOR, TerminalBlock_4Ucon:TerminalBlock_4Ucon_1x03_P3.50mm_Horizontal, F.Cu at (245.7, 106.5)
- added P51: CONN_SENSOR, TerminalBlock_4Ucon:TerminalBlock_4Ucon_1x03_P3.50mm_Horizontal, F.Cu at (233.4, 106.5)
- added R198: RES_470R_1%_0402, Resistor_SMD:R_0402_1005Metric, F.Cu at (239.6, 112.8)
- added R199: RES_10K_1%_0402, Resistor_SMD:R_0402_1005Metric, F.Cu at (242.6, 112.7)
- added R200: RES_NTC_10K_402, Resistor_SMD:R_0402_1005Metric, F.Cu at (245.6, 111.2)
- added R201: RES_10K_1%_0402, Resistor_SMD:R_0402_1005Metric, F.Cu at (256.1, 103.1)
- added R202: RES_NTC_10K_402, Resistor_SMD:R_0402_1005Metric, F.Cu at (256.1, 104.1)
- added U36: IC_TXS0108, Package_SO:TSSOP-20_4.4x6.5mm_P0.65mm, F.Cu at (234.8, 114.2)
- moved P45 14.6 mm to (267.1, -58.3)
Connections:
- C102 pad 1: Net-(C102-Pad1) -> VDD_3V3
- C103 pad 1: Net-(C100-Pad1) -> Net-(C103-Pad1)
- C104 pad 1: Net-(C101-Pad1) -> Net-(C104-Pad1)
- C111 pad 1: Net-(C102-Pad1) -> VDD_3V3
- C112 pad 2: GND -> Net-(C103-Pad1)
- C113 pad 2: GND -> Net-(C104-Pad1)
- C93 pad 1: Net-(C102-Pad1) -> VDD_3V3
- C95 pad 1: Net-(C102-Pad1) -> VDD_3V3
- C96 pad 1: Net-(C102-Pad1) -> VDD_3V3
- C99 pad 1: Net-(C102-Pad1) -> VDD_3V3
- U12 pad 110: Net-(U12-Pad110) -> GPEX_CS
- U12 pad 15: OC_ADJ1 -> TEMP_MOT1
- U12 pad 18: OC_ADJ2 -> PWM_IN1
- U12 pad 19: GPEX_CS -> PWM_IN2
- U12 pad 20: GPEX_RESET -> TEMP_MOT2
- U12 pad 49: Net-(U12-Pad49) -> OC_ADJ2
- U12 pad 7: Net-(U12-Pad7) -> OC_ADJ1
- U12 pad 8: Net-(U12-Pad8) -> GPEX_RESET

Commit message: start component placement
Parts:
- removed C153: CAP_100nF_50V_0402, Capacitor_SMD:C_0402_1005Metric
- removed P50, P51: CONN_SENSOR, TerminalBlock_4Ucon:TerminalBlock_4Ucon_1x03_P3.50mm_Horizontal
- added C158: CAP_2.2uF_16V_0402, Capacitor_SMD:C_0402_1005Metric, F.Cu at (251.1, 143.3)
- added C159: CAP_2.2uF_16V_0402, Capacitor_SMD:C_0402_1005Metric, F.Cu at (249.1, 145.4)
- added C160: CAP_2.2uF_16V_0402, Capacitor_SMD:C_0402_1005Metric, F.Cu at (255.7, 139.2)
- added C161: CAP_2.2uF_16V_0402, Capacitor_SMD:C_0402_1005Metric, F.Cu at (257.8, 137.2)
- added C162: CAP_2.2uF_16V_0402, Capacitor_SMD:C_0402_1005Metric, F.Cu at (253.1, 142.3)
- added C163: CAP_2.2uF_16V_0402, Capacitor_SMD:C_0402_1005Metric, F.Cu at (246.3, 147.4)
- added C164: CAP_2.2uF_16V_0402, Capacitor_SMD:C_0402_1005Metric, F.Cu at (257.8, 138.2)
- added C165: CAP_2.2uF_100V_1210, Capacitor_SMD:C_1210_3225Metric, F.Cu at (238.6, 138.2)
- added C166: CAP_100pF_50V_0402, Capacitor_SMD:C_0402_1005Metric, F.Cu at (251.1, 144.3)
- added C167: CAP_2.2uF_100V_1210, Capacitor_SMD:C_1210_3225Metric, F.Cu at (241.2, 134.5)
- added C168: CAP_2.2uF_16V_0402, Capacitor_SMD:C_0402_1005Metric, F.Cu at (248.0, 147.4)
- added C169: CAPP_100uF_25V_6357, Capacitor_SMD:CP_Elec_6.3x5.7, F.Cu at (231.5, 140.0)
- added C170: CAP_2.2uF_16V_0402, Capacitor_SMD:C_0402_1005Metric, F.Cu at (253.1, 141.3)
- added C171: CAP_2.2uF_16V_0402, Capacitor_SMD:C_0402_1005Metric, F.Cu at (254.0, 140.2)
- added D32: D_BAT54, Diode_SMD:D_SOD-123, F.Cu at (229.2, 144.6)
- added D33: D_BAT54, Diode_SMD:D_SOD-123, F.Cu at (241.3, 131.7)
- added F1: FUSE_3A_9750, CUSTOM:Fuse_Littlefuse_9750, F.Cu at (232.9, 133.5)
- added F2: FUSE_4A_0603, Fuse:Fuse_0603_1608Metric, F.Cu at (228.3, 146.5)
- added R203: RES_10K_1%_0402, Resistor_SMD:R_0402_1005Metric, F.Cu at (249.4, 143.3)
- added R204: RES_10K_1%_0402, Resistor_SMD:R_0402_1005Metric, F.Cu at (244.6, 147.4)
- added R205: RES_10K_1%_0402, Resistor_SMD:R_0402_1005Metric, F.Cu at (242.9, 147.4)
- added R206: RES_10K_1%_0402, Resistor_SMD:R_0402_1005Metric, F.Cu at (232.7, 148.0)
- added R207: RES_10K_1%_0402, Resistor_SMD:R_0402_1005Metric, F.Cu at (249.4, 144.3)
- added R208: RES_10K_1%_0402, Resistor_SMD:R_0402_1005Metric, F.Cu at (251.4, 142.3)
- added R209: RES_270R_1%_0402, Resistor_SMD:R_0402_1005Metric, F.Cu at (227.6, 147.8)
- added R210: RES_270R_1%_0402, Resistor_SMD:R_0402_1005Metric, F.Cu at (256.1, 138.2)
- added R211: RES_270R_1%_0402, Resistor_SMD:R_0402_1005Metric, F.Cu at (251.4, 141.3)
- added R212: RES_270R_1%_0402, Resistor_SMD:R_0402_1005Metric, F.Cu at (256.1, 137.2)
- added R213: RES_270R_1%_0402, Resistor_SMD:R_0402_1005Metric, F.Cu at (254.0, 139.2)
- added TP100: Test_Point, CUSTOM:TestPoint_Pad_0.5x0.5mm, F.Cu at (248.6, 135.6)
- added TP101: Test_Point, CUSTOM:TestPoint_Pad_0.5x0.5mm, F.Cu at (103.0, -0.50)
- added TP102: Test_Point, CUSTOM:TestPoint_Pad_0.5x0.5mm, F.Cu at (92.2, 4.00)
- added TP42: Test_Point, CUSTOM:TestPoint_Pad_0.5x0.5mm, F.Cu at (243.1, 145.9)
- added TP43: Test_Point, CUSTOM:TestPoint_Pad_0.5x0.5mm, F.Cu at (250.1, 139.7)
- added TP44: Test_Point, CUSTOM:TestPoint_Pad_0.5x0.5mm, F.Cu at (252.2, 137.7)
- added TP45: Test_Point, CUSTOM:TestPoint_Pad_0.5x0.5mm, F.Cu at (254.8, 135.6)
- added TP46: Test_Point, CUSTOM:TestPoint_Pad_0.5x0.5mm, F.Cu at (257.0, 133.6)
- added TP47: Test_Point, CUSTOM:TestPoint_Pad_0.5x0.5mm, F.Cu at (245.1, 145.9)
- added TP48: Test_Point, CUSTOM:TestPoint_Pad_0.5x0.5mm, F.Cu at (247.5, 143.8)
- added TP49: Test_Point, CUSTOM:TestPoint_Pad_0.5x0.5mm, F.Cu at (249.6, 141.8)
- added TP50: Test_Point, CUSTOM:TestPoint_Pad_0.5x0.5mm, F.Cu at (254.2, 137.7)
- added TP51: Test_Point, CUSTOM:TestPoint_Pad_0.5x0.5mm, F.Cu at (250.8, 133.6)
- added TP52: Test_Point, CUSTOM:TestPoint_Pad_0.5x0.5mm, F.Cu at (243.4, 143.8)
- added TP53: Test_Point, CUSTOM:TestPoint_Pad_0.5x0.5mm, F.Cu at (245.5, 141.8)
- added TP54: Test_Point, CUSTOM:TestPoint_Pad_0.5x0.5mm, F.Cu at (248.8, 131.5)
- added TP55: Test_Point, CUSTOM:TestPoint_Pad_0.5x0.5mm, F.Cu at (250.7, 135.6)
- added TP56: Test_Point, CUSTOM:TestPoint_Pad_0.5x0.5mm, F.Cu at (252.9, 133.6)
- added TP57: Test_Point, CUSTOM:TestPoint_Pad_0.5x0.5mm, F.Cu at (254.9, 131.5)
- added TP58: Test_Point, CUSTOM:TestPoint_Pad_0.5x0.5mm, F.Cu at (241.0, 145.3)
- added TP59: Test_Point, CUSTOM:TestPoint_Pad_0.5x0.5mm, F.Cu at (239.0, 147.0)
- added TP60: Test_Point, CUSTOM:TestPoint_Pad_0.5x0.5mm, F.Cu at (248.1, 137.7)
- added TP61: Test_Point, CUSTOM:TestPoint_Pad_0.5x0.5mm, F.Cu at (243.4, 141.8)
- added TP62: Test_Point, CUSTOM:TestPoint_Pad_0.5x0.5mm, F.Cu at (248.8, 133.6)
- added TP63: Test_Point, CUSTOM:TestPoint_Pad_0.5x0.5mm, F.Cu at (248.1, 139.7)
- added TP64: Test_Point, CUSTOM:TestPoint_Pad_0.5x0.5mm, F.Cu at (247.2, 145.9)
- added TP65: Test_Point, CUSTOM:TestPoint_Pad_0.5x0.5mm, F.Cu at (247.5, 141.8)
- added TP66: Test_Point, CUSTOM:TestPoint_Pad_0.5x0.5mm, F.Cu at (245.5, 143.8)
- added TP67: Test_Point, CUSTOM:TestPoint_Pad_0.5x0.5mm, F.Cu at (110.2, 5.00)
- added TP68: Test_Point, CUSTOM:TestPoint_Pad_0.5x0.5mm, F.Cu at (110.2, 4.00)
- added TP69: Test_Point, CUSTOM:TestPoint_Pad_0.5x0.5mm, F.Cu at (110.2, 6.00)
- added TP70: Test_Point, CUSTOM:TestPoint_Pad_0.5x0.5mm, F.Cu at (110.2, 7.00)
- added TP71: Test_Point, CUSTOM:TestPoint_Pad_0.5x0.5mm, F.Cu at (110.2, 8.00)
- added TP72: Test_Point, CUSTOM:TestPoint_Pad_0.5x0.5mm, F.Cu at (110.2, 9.00)
- added TP73: Test_Point, CUSTOM:TestPoint_Pad_0.5x0.5mm, F.Cu at (187.8, -36.8)
- added TP74: Test_Point, CUSTOM:TestPoint_Pad_0.5x0.5mm, F.Cu at (187.8, -35.8)
- added TP75: Test_Point, CUSTOM:TestPoint_Pad_0.5x0.5mm, F.Cu at (244.5, 135.6)
- added TP76: Test_Point, CUSTOM:TestPoint_Pad_0.5x0.5mm, F.Cu at (234.9, 147.0)
- added TP77: Test_Point, CUSTOM:TestPoint_Pad_0.5x0.5mm, F.Cu at (244.0, 137.7)
- added TP78: Test_Point, CUSTOM:TestPoint_Pad_0.5x0.5mm, F.Cu at (246.6, 135.6)
- added TP79: Test_Point, CUSTOM:TestPoint_Pad_0.5x0.5mm, F.Cu at (239.3, 140.8)
- added TP80: Test_Point, CUSTOM:TestPoint_Pad_0.5x0.5mm, F.Cu at (256.8, 135.6)
- added TP81: Test_Point, CUSTOM:TestPoint_Pad_0.5x0.5mm, F.Cu at (250.1, 137.7)
- added TP82: Test_Point, CUSTOM:TestPoint_Pad_0.5x0.5mm, F.Cu at (252.2, 139.7)
- added TP83: Test_Point, CUSTOM:TestPoint_Pad_0.5x0.5mm, F.Cu at (241.9, 139.2)
- added TP84: Test_Point, CUSTOM:TestPoint_Pad_0.5x0.5mm, F.Cu at (241.4, 141.2)
- added TP85: Test_Point, CUSTOM:TestPoint_Pad_0.5x0.5mm, F.Cu at (239.3, 142.9)
- added TP86: Test_Point, CUSTOM:TestPoint_Pad_0.5x0.5mm, F.Cu at (236.7, 144.9)
- added TP87: Test_Point, CUSTOM:TestPoint_Pad_0.5x0.5mm, F.Cu at (117.2, -3.75)
- added TP88: Test_Point, CUSTOM:TestPoint_Pad_0.5x0.5mm, F.Cu at (117.2, -5.75)
- added TP89: Test_Point, CUSTOM:TestPoint_Pad_0.5x0.5mm, F.Cu at (232.8, 146.5)
- added TP90: Test_Point, CUSTOM:TestPoint_Pad_0.5x0.5mm, F.Cu at (237.3, 142.9)
- added TP91: Test_Point, CUSTOM:TestPoint_Pad_0.5x0.5mm, F.Cu at (244.7, 133.6)
- added TP92: Test_Point, CUSTOM:TestPoint_Pad_0.5x0.5mm, F.Cu at (246.7, 131.5)
- added TP93: Test_Point, CUSTOM:TestPoint_Pad_0.5x0.5mm, F.Cu at (234.6, 144.4)
- added TP94: Test_Point, CUSTOM:TestPoint_Pad_0.5x0.5mm, F.Cu at (241.9, 137.1)
- added TP95: Test_Point, CUSTOM:TestPoint_Pad_0.5x0.5mm, F.Cu at (230.8, 146.8)
- added TP96: Test_Point, CUSTOM:TestPoint_Pad_0.5x0.5mm, F.Cu at (187.8, -34.8)
- added TP97: Test_Point, CUSTOM:TestPoint_Pad_0.5x0.5mm, F.Cu at (252.9, 131.5)
- added TP98: Test_Point, CUSTOM:TestPoint_Pad_0.5x0.5mm, F.Cu at (246.0, 139.7)
- added TP99: Test_Point, CUSTOM:TestPoint_Pad_0.5x0.5mm, F.Cu at (246.7, 133.6)
- C102, C114, C118, C63, C82, C83, C95, C96, C99: value CAP_100nF_100V_0603 -> CAP_100nF_50V_0402; footprint Capacitor_SMD:C_0603_1608Metric -> Capacitor_SMD:C_0402_1005Metric
- C111, C117, C119, C151, C86, C93: value CAP_100nF_100V_0603 -> CAP_100nF_50V_0402; footprint Capacitor_SMD:C_0603_1608Metric -> Capacitor_SMD:C_0402_1005Metric; moved to B.Cu
- C13: value CAP_100nF_50V_0402 -> CAP_2.2uF_16V_0402
- C141, C142: value CAP_2.2nF_50V_0603 -> CAP_22nF_50V_0402; footprint Capacitor_SMD:C_0603_1608Metric -> Capacitor_SMD:C_0402_1005Metric
- C147, C148: value CAP_2.2uF_100V_1210 -> CAP_2.2uF_16V_0402; footprint Capacitor_SMD:C_1210_3225Metric -> Capacitor_SMD:C_0402_1005Metric
- C152: value CAP_100nF_50V_0402 -> CAP_22uF_10V_0805; footprint Capacitor_SMD:C_0402_1005Metric -> Capacitor_SMD:C_0805_2012Metric
- C19: value CAP_51pF_50V_0402 -> CAP_100pF_50V_0402
- C45: value CAP_10uF_35V_0603 -> CAP_10uF_25V_0805; footprint Capacitor_SMD:C_0603_1608Metric -> Capacitor_SMD:C_0805_2012Metric
- C49: value CAP_100nF_50V_0402 -> CAP_10uF_25V_0805; footprint Capacitor_SMD:C_0402_1005Metric -> Capacitor_SMD:C_0805_2012Metric
- C87, C88, C91, C92: value CAP_1uF_10V_0402 -> CAP_2.2uF_16V_0402
- D10, D11, D13: value D_ESDCAN06 -> D_ESDCAN03
- D15: value D_MM3Z3V3B -> D_BAT54; footprint Diode_SMD:D_SOD-323F -> Diode_SMD:D_SOD-123
- D16: value D_MM3Z3V3B -> D_SZ1SMB5913BT3G; footprint Diode_SMD:D_SOD-323F -> Diode_SMD:D_SMB
- D30: value D_BAT54 -> D_SZ1SMB5913BT3G; footprint Diode_SMD:D_SOD-123 -> Diode_SMD:D_SMB
- FB2, FB3, R108, R110, R77: moved to B.Cu
- J1: footprint Connector_USB:USB_Micro-B_GCT_USB3076-30-A -> CUSTOM:USB_Micro-B_GCT_USB3076-30-A
- J2, J3: footprint Connector_RJ:RJ45_Tranformer -> CUSTOM:RJ45_Tranformer
- L1: value L_100uH_3.64A -> L_33uH_4.2A_45mR
- P1, P2, P3, P4, P5, P6, P7, P8: footprint TerminalBlock_4Ucon:TerminalBlock_4Ucon_1x02_P3.50mm_Horizontal -> CUSTOM:CONN_SWITCH
- P10, P11, P12, P13, P14, P15, P16, P38, P39, P40, P42, P43, P44, P9: footprint TerminalBlock_4Ucon:TerminalBlock_4Ucon_1x03_P3.50mm_Horizontal -> CUSTOM:CONN_SENSOR
- P17: footprint Connector_PinSocket_2.54mm:PinSocket_2x05_P2.54mm_Vertical -> Connector_IDC:IDC-Header_2x05_P2.54mm_Vertical
- P19, P20, P24: footprint TerminalBlock_4Ucon:TerminalBlock_4Ucon_1x03_P3.50mm_Horizontal -> CUSTOM:CONN_CAN
- P21, P22, P26, P27: footprint TerminalBlock_4Ucon:TerminalBlock_4Ucon_1x02_P3.50mm_Horizontal -> CUSTOM:CONN_AN_OUT
- P23: footprint TerminalBlock_4Ucon:TerminalBlock_4Ucon_1x02_P3.50mm_Horizontal -> CUSTOM:CONN_POWER_10A
- P25: footprint Connector_PinSocket_2.54mm:PinSocket_2x08_P2.54mm_Vertical -> CUSTOM:CONN_LCD
- P28: footprint Connector_PinSocket_2.54mm:PinSocket_2x05_P2.54mm_Vertical -> CUSTOM:CONN_UEXT
- P29, P30, P31, P32, P33, P34, P35, P36: footprint TerminalBlock_4Ucon:TerminalBlock_4Ucon_1x02_P3.50mm_Horizontal -> CUSTOM:CONN_LED
- P47, P48: footprint TerminalBlock_MetzConnect:TerminalBlock_MetzConnect_Type059_RT06305HBWC_1x05_P3.50mm_Horizontal -> CUSTOM:CONN_HALL
- P49: footprint TerminalBlock_4Ucon:TerminalBlock_4Ucon_1x02_P3.50mm_Horizontal -> CUSTOM:CONN_BRKRES
- Q1, Q2, Q3, Q4, Q5, Q6: value Q_NMOS_2X_100V_70A -> Q_NMOS_2X_60V_63A
- R109: value RES_10K_1%_0402 -> RES_270R_1%_0402
- R114, R115, R150, R151: footprint CUSTOM:WSLF25123L000FEA -> CUSTOM:R_2818_7146Metric
- R117, R119, R156, R158, R189, R191, R68: value RES_135K_1%_0402 -> RES_137K_1%_0402
- R121, R122, R161, R162: value RES_22R_1%_0402 -> RES_270R_1%_0402
- R123, R124, R125, R126, R127, R128, R145, R146: value RES_49.9_0.1%_0805 -> RES_49.9_0.1%_0402; footprint Resistor_SMD:R_0805_2012Metric -> Resistor_SMD:R_0402_1005Metric
- R196, R197: value RES_135K_1%_0402 -> RES_10K_1%_0402
- R34, R43, R44, R63, R64: value RES_0R_0402 -> RES_10K_1%_0402
- R35: value RES_0R_0402 -> RES_147k_1%_0603; footprint Resistor_SMD:R_0402_1005Metric -> Resistor_SMD:R_0603_1608Metric
- R36, R45: value RES_0R_0402 -> RES_3K_1%_0402
- R37: value RES_5K_1%_0402 -> RES_3K_1%_0402
- R40: value RES_1M_1%_0402 -> RES_137K_1%_0402
- R48: value RES_147k_1%_0603 -> RES_137K_1%_0402; footprint Resistor_SMD:R_0603_1608Metric -> Resistor_SMD:R_0402_1005Metric
- R49: value RES_10.5k_1%_0603 -> RES_10K_1%_0402; footprint Resistor_SMD:R_0603_1608Metric -> Resistor_SMD:R_0402_1005Metric
- R59: value RES_24k_1%_0603 -> RES_3K_1%_0402; footprint Resistor_SMD:R_0603_1608Metric -> Resistor_SMD:R_0402_1005Metric
- R65: value RES_10mOhm_1% -> RES_0R_0402; footprint Resistor_SMD:R_0805_2012Metric -> Resistor_SMD:R_0402_1005Metric
- R66: value RES_10K_1%_0402 -> RES_10mOhm_1%; footprint Resistor_SMD:R_0402_1005Metric -> Resistor_SMD:R_0805_2012Metric
- R76: value RES_22R_1%_0402 -> RES_10mOhm_1%; footprint Resistor_SMD:R_0402_1005Metric -> Resistor_SMD:R_0805_2012Metric
- R78, R79: value RES_135K_1%_0402 -> RES_270R_1%_0402
- R80, R81, R82, R83: value RES_1K5_1%_0402 -> RES_3K_1%_0402
- S1: footprint SOIC:SOIC127P670X145-8N -> CUSTOM:SW_PTS540
- TP1, TP10, TP11, TP12, TP13, TP14, TP15, TP16, TP17, TP18, TP19, TP2, TP20, TP21, TP22, TP23, TP24, TP25, TP26, TP27, TP28, TP29, TP3, TP30, TP31, TP32, TP33, TP34, TP35, TP36, TP37, TP38, TP39, TP4, TP40, TP41, TP5, TP6, TP7, TP8, TP9: footprint TestPoint:TestPoint_Pad_1.0x1.0mm -> CUSTOM:TestPoint_Pad_0.5x0.5mm
- U14: footprint SOIC:SOIC127P600X175_HS-9N -> CUSTOM:TI_SO-PowerPAD-8
- U18, U27, U28: footprint Package_TO_SOT_SMD:SOT-23-6 -> CUSTOM:SOT-23-6L
- U20, U22: value IC_TLV5533 -> IC_TLV75533
- U21: footprint Package_DFN_QFN:WQFN-24-1EP_4x4mm_P0.5mm_EP2.7x2.7mm -> CUSTOM:WQFN-24-1EP_4x4mm_P0.5mm_EP2.7x2.7mm_Thermal
- U30: value LAN9252 -> IC_LAN9252; footprint CUSTOM:TQFP-64-1EP_10x10mm_P0.5mm_EP6x6mm -> TQFP-64-1EP_10x10mm_P0.5mm_EP5.7x5.7mm
- U36: value IC_TXS0108 -> IC_TLV75533; footprint Package_SO:TSSOP-20_4.4x6.5mm_P0.65mm -> Package_TO_SOT_SMD:SOT-23-5
- Y1: footprint Crystal:Crystal_SMD_5032-4Pin_5.0x3.2mm -> CUSTOM:Crystal_ABM3B_5032-4Pin_5.0x3.2mm
- Y2, Y3: footprint Crystal:Crystal_SMD_3225-4Pin_3.2x2.5mm -> CUSTOM:Crystal_SMD_3225-4Pin_3.2x2.5mm
- moved J2 212.5 mm to (86.9, -37.1)
- moved J3 212.3 mm to (106.8, -37.1)
- moved C129 208.1 mm to (224.8, -54.2), turned to 180 degrees
- moved R178 193.8 mm to (204.2, -50.5), turned to 180 degrees
- moved R179 192.1 mm to (204.2, -51.5)
- moved C151 190.9 mm to (92.0, -5.00)
- moved R131 186.9 mm to (204.2, -47.0)
- moved R133 185.5 mm to (204.2, -45.0)
- moved C140 182.6 mm to (230.5, -59.0), turned to 90 degrees
- moved C133 179.4 mm to (224.8, -40.5), turned to 180 degrees
- moved R199 174.5 mm to (213.0, -59.2)
- moved C154 174.2 mm to (209.2, -56.8)
- moved C97 173.6 mm to (194.8, -48.2)
- moved C143 172.9 mm to (230.5, -11.5), turned to 270 degrees
- moved C156 171.5 mm to (211.8, -54.2)
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Connections:
- net BREAK renamed VMOT_IN
- net ENCIRQ2 renamed MOTOR2_BRKIN
- C100 pad 1: Net-(C100-Pad1) -> VMOT
- C101 pad 1: Net-(C101-Pad1) -> VMOT
- C11 pad 2: AIN_VDD_5V -> USB_5V
- C112 pad 1: Net-(C100-Pad1) -> VMOT
- C113 pad 1: Net-(C101-Pad1) -> VMOT
- C12 pad 2: AIN_VDD_5V -> USB_5V
- C124 pad 1: VSA2 -> VSA2_RAW
- C146 pad 1: VSB2 -> VSB2_RAW
- C147 pad 1: USB_5V -> ENC2VDD5V
- C148 pad 1: USB_5V -> ENC1VDD5V
- C150 pad 1: VSC2 -> VSC2_RAW
- C152 pad 1: VDD_3V3 -> Net-(C152-Pad1)
- C16 pad 1: Net-(C16-Pad1) -> VREF1
- C28 pad 1: VDD_3V3 -> VDD_3V3_MCU
- C29 pad 1: VDD_3V3 -> VDD_3V3_MCU
- C3 pad 1: VDD_3V3 -> VDD_3V3_MCU
- C32 pad 1: VDD_3V3 -> Net-(C32-Pad1)
- C34 pad 1: VDD_3V3 -> VDD_3V3_MCU
- C35 pad 1: VDD_3V3 -> VDD_3V3_MCU
- C38 pad 1: Net-(C38-Pad1) -> Net-(C168-Pad1)
- C39 pad 1: VDD_3V3 -> VDD_3V3_MCU
- C40 pad 1: VDD_3V3 -> VDD_3V3_MCU
- C41 pad 1: VDD_3V3 -> VDD_3V3_MCU
- C42 pad 1: VDD_3V3 -> VDD_3V3_MCU
- C43 pad 1: VDD_3V3 -> VDD_3V3_MCU
- C44 pad 1: VDD_3V3 -> VDD_3V3_MCU
- C45 pad 1: Net-(C45-Pad1) -> Net-(C169-Pad1)
- C47 pad 1: VDD_3V3 -> VDD_3V3_MCU
- C48 pad 1: VDD_3V3 -> VDD_3V3_MCU
- C50 pad 1: VDD_3V3 -> Net-(C32-Pad1)
- C51 pad 1: VDD_3V3 -> AIN_VDD_5V
- C52 pad 1: USB_5V -> Net-(C52-Pad1)
- C55 pad 1: USB_5V -> Net-(C52-Pad1)
- C59 pad 1: VDD_3V3 -> VDD_3V3_MCU
- C60 pad 1: VDD_3V3 -> VDD_3V3_MCU
- D1 pad 2: AIN_VDD_5V -> USB_5V
- D14 pad 1: Net-(C38-Pad1) -> Net-(D14-Pad1)
- D15 pad 1: Net-(C54-Pad1) -> Net-(D15-Pad1)
- D15 pad 2: GND -> MOTOR1_BRKIN
- D16 pad 1: VDD_3V3 -> Net-(C58-Pad1)
- D2 pad 2: AIN_VDD_5V -> USB_5V
- D20 pad 3: VSA2 -> VSA2_RAW
- D22 pad 3: VSB2 -> VSB2_RAW
- D23 pad 3: (no net) -> GND
- D23 pad 4: GND -> HALL_C1
- D24 pad 3: (no net) -> GND
- D24 pad 4: GND -> HALL_C2
- D26 pad 3: VSC2 -> VSC2_RAW
- D3 pad 2: AIN_VDD_5V -> USB_5V
- D30 pad 1: Net-(D30-Pad1) -> Net-(C152-Pad1)
- D4 pad 2: AIN_VDD_5V -> USB_5V
- D5 pad 2: AIN_VDD_5V -> USB_5V
- D6 pad 2: AIN_VDD_5V -> USB_5V
- D7 pad 2: AIN_VDD_5V -> USB_5V
- D8 pad 2: AIN_VDD_5V -> USB_5V
- FB1 pad 1: Net-(C16-Pad1) -> VREF1
- FB1 pad 2: VREF1 -> Net-(C32-Pad1)
- J1 pad 1: USB_5V -> Net-(J1-Pad1)
- L1 pad 2: Net-(C38-Pad1) -> Net-(C168-Pad1)
- L2 pad 2: USB_5V -> Net-(C52-Pad1)
- P23 pad 1: Net-(C45-Pad1) -> Net-(F1-Pad2)
- P45 pad 1: SLA1 -> SLC1
- P45 pad 3: SLC1 -> SLA1
- P46 pad 1: SLA2 -> SLC2
- P46 pad 3: SLC2 -> SLA2
- P47 pad 4: USB_5V -> ENC1VDD5V
- P48 pad 4: USB_5V -> ENC2VDD5V
- Q8 pad 1: Net-(D30-Pad1) -> Net-(Q8-Pad1)
- R109 pad 1: GND -> GPIO_SCK
- R111 pad 1: Net-(R111-Pad1) -> VSA1
- R112 pad 1: Net-(R112-Pad1) -> VSA2
- R119 pad 2: VSA2 -> VSA2_RAW
- R120 pad 2: VSA2 -> VSA2_RAW
- R121 pad 1: VSA1 -> ENCMISO1
- R121 pad 2: Net-(R111-Pad1) -> Net-(R121-Pad2)
- R122 pad 1: VSA2 -> ENCMISO2
- R122 pad 2: Net-(R112-Pad1) -> Net-(R121-Pad2)
- R152 pad 1: Net-(J3-PadGA) -> Net-(J3-Pad10)
- R153 pad 1: Net-(R153-Pad1) -> VSB1
- R154 pad 1: Net-(R154-Pad1) -> VSB2
- R155 pad 1: Net-(J2-PadGA) -> Net-(J2-Pad10)
- R158 pad 2: VSB2 -> VSB2_RAW
- R159 pad 2: VSB2 -> VSB2_RAW
- R161 pad 1: VSB1 -> GPIO_MISO
- R161 pad 2: Net-(R153-Pad1) -> Net-(R121-Pad2)
- R162 pad 1: VSB2 -> ENCMOSI1
- R162 pad 2: Net-(R154-Pad1) -> Net-(R162-Pad2)
- R163 pad 1: HALL_A1 -> Net-(P47-Pad1)
- R163 pad 2: GND -> HALL_A1
- R164 pad 1: HALL_A2 -> Net-(P48-Pad1)
- R164 pad 2: GND -> HALL_A2
- R165 pad 1: HALL_B1 -> Net-(P47-Pad3)
- R165 pad 2: GND -> HALL_C1
- R166 pad 1: HALL_B2 -> Net-(P48-Pad2)
- R166 pad 2: GND -> HALL_B2
- R167 pad 1: HALL_C1 -> Net-(P47-Pad2)
- R167 pad 2: GND -> HALL_B1
- R168 pad 1: HALL_C2 -> Net-(P48-Pad3)
- R168 pad 2: GND -> HALL_C2
- R183 pad 1: Net-(P47-Pad1) -> GND
- R184 pad 1: Net-(P47-Pad2) -> GND
- R185 pad 1: Net-(P47-Pad3) -> GND
- R186 pad 1: Net-(P48-Pad1) -> GND
- R187 pad 1: Net-(P48-Pad2) -> GND
- R188 pad 1: Net-(P48-Pad3) -> GND
- R191 pad 2: VSC2 -> VSC2_RAW
- R192 pad 2: VSC2 -> VSC2_RAW
- R196 pad 1: Net-(D30-Pad1) -> Net-(Q8-Pad1)
- R197 pad 1: Net-(D30-Pad1) -> Net-(Q8-Pad1)
- R34 pad 1: Net-(R34-Pad1) -> AIN_OC
- R34 pad 2: GND -> VDD_3V3_MCU
- R35 pad 1: Net-(R35-Pad1) -> Net-(C52-Pad1)
- R35 pad 2: GND -> Net-(R35-Pad2)
- R36 pad 1: Net-(R36-Pad1) -> AP_SDA1
- R36 pad 2: GND -> VDD_3V3_MCU
- R43 pad 1: Net-(R43-Pad1) -> VDD_3V3_MCU
- R43 pad 2: GND -> ENCOC1
- R44 pad 1: Net-(R44-Pad1) -> VDD_3V3_MCU
- R44 pad 2: GND -> ENCOC2
- R45 pad 1: Net-(R45-Pad1) -> AP_SCL1
- R45 pad 2: GND -> VDD_3V3_MCU
- R48 pad 1: Net-(C38-Pad1) -> Net-(C168-Pad1)
- R55 pad 1: Net-(C38-Pad1) -> Net-(D14-Pad1)
- R55 pad 2: Net-(C45-Pad1) -> Net-(C169-Pad1)
- R58 pad 1: USB_5V -> Net-(C52-Pad1)
- R59 pad 1: Net-(R58-Pad2) -> Net-(R59-Pad1)
- R59 pad 2: GND -> Net-(R58-Pad2)
- R61 pad 1: Net-(R61-Pad1) -> USB_5V
- R61 pad 2: USB_5V -> Net-(C52-Pad1)
- R63 pad 1: GND -> Net-(R63-Pad1)
- R63 pad 2: Net-(R63-Pad2) -> Net-(R59-Pad1)
- R64 pad 1: GND -> Net-(R63-Pad1)
- R64 pad 2: Net-(R64-Pad2) -> GND
- R65 pad 1: VDD_3V3 -> USB_5V
- R65 pad 2: Net-(C58-Pad1) -> Net-(J1-Pad1)
- R66 pad 1: Net-(R66-Pad1) -> VDD_3V3
- R66 pad 2: VDD_3V3 -> Net-(C58-Pad1)
- R76 pad 1: VMOT_SENSE -> VDD_3V3_MCU
- R76 pad 2: Net-(R76-Pad2) -> Net-(C152-Pad1)
- R78 pad 1: OC_ADJ1 -> ENCSCK1
- R78 pad 2: VDD_3V3 -> Net-(R109-Pad2)
- R79 pad 1: OC_ADJ2 -> ENCSCK2
- R79 pad 2: VDD_3V3 -> Net-(R109-Pad2)
- R84 pad 2: VDD_3V3 -> VDD_3V3_MCU
- R85 pad 2: VDD_3V3 -> VDD_3V3_MCU
- R86 pad 2: VDD_3V3 -> VDD_3V3_MCU
- R87 pad 2: VDD_3V3 -> VDD_3V3_MCU
- TP16 pad 1: Net-(C45-Pad1) -> Net-(C169-Pad1)
- TP17 pad 1: Net-(C38-Pad1) -> Net-(D14-Pad1)
- TP18 pad 1: Net-(TP18-Pad1) -> Net-(R35-Pad2)
- TP19 pad 1: USB_5V -> Net-(C52-Pad1)
- TP20 pad 1: Net-(R61-Pad1) -> USB_5V
- TP22 pad 1: VDD_3V3 -> SW1
- TP38 pad 1: OC_ADJ1 -> OC_ADJ2
- TP39 pad 1: Net-(R81-Pad2) -> Net-(R80-Pad2)
- TP40 pad 1: Net-(R83-Pad2) -> Net-(R82-Pad2)
- TP41 pad 1: Net-(D30-Pad1) -> Net-(Q8-Pad1)
- U11 pad 1: Net-(U11-Pad1) -> Net-(TP56-Pad1)
- U11 pad 2: Net-(U11-Pad2) -> Net-(TP57-Pad1)
- U12 pad 108: VDD_3V3 -> VDD_3V3_MCU
- U12 pad 110: GPEX_CS -> ENCA1
- U12 pad 111: ENCSCK1 -> Net-(R109-Pad2)
- U12 pad 112: ENCMISO1 -> Net-(R121-Pad2)
- U12 pad 113: ENCMOSI1 -> Net-(R162-Pad2)
- U12 pad 121: VDD_3V3 -> VDD_3V3_MCU
- U12 pad 122: ENCSG1 -> FAULT1
- U12 pad 123: ENCSY1 -> FAULT2
- U12 pad 131: VDD_3V3 -> VDD_3V3_MCU
- U12 pad 136: HALL_C1 -> GPEX_CS
- U12 pad 143: VDD_3V3 -> VDD_3V3_MCU
- U12 pad 144: VDD_3V3 -> VDD_3V3_MCU
- U12 pad 17: VDD_3V3 -> VDD_3V3_MCU
- U12 pad 26: VSB1 -> VSA1
- U12 pad 27: VSC1 -> VSB1
- U12 pad 28: VSA2 -> VSC1
- U12 pad 29: VSB2 -> VSA2
- U12 pad 30: VDD_3V3 -> VDD_3V3_MCU
- U12 pad 32: VREF1 -> Net-(C32-Pad1)
- U12 pad 33: VREF1 -> Net-(C32-Pad1)
- U12 pad 39: VDD_3V3 -> VDD_3V3_MCU
- U12 pad 41: ENCA1 -> SOA2
- U12 pad 44: VSC2 -> VSB2
- U12 pad 45: VSA1 -> VSC2
- U12 pad 46: SOA2 -> HALL_C1
- U12 pad 49: OC_ADJ2 -> GPEX_RESET
- U12 pad 52: VDD_3V3 -> VDD_3V3_MCU
- U12 pad 6: VDD_3V3 -> VDD_3V3_MCU
- U12 pad 62: VDD_3V3 -> VDD_3V3_MCU
- U12 pad 68: ENCIRQ1 -> MOTOR1_BRKIN
- U12 pad 7: OC_ADJ1 -> POTADDRA
- U12 pad 72: VDD_3V3 -> VDD_3V3_MCU
- U12 pad 77: ENCSH2 -> ENCZ1
- U12 pad 78: ENCSG2 -> OCW1
- U12 pad 79: ENCSY2 -> OCW2
- U12 pad 8: GPEX_RESET -> POTADDRB
- U12 pad 80: ENCCS2 -> ENCSH2
- U12 pad 84: VDD_3V3 -> VDD_3V3_MCU
- U12 pad 86: ENCZ1 -> ENCCS2
- U12 pad 89: CAN_STB1 -> DC_CAL1
- U12 pad 9: Net-(U12-Pad9) -> POTADDRC
- U12 pad 90: CAN_STB2 -> DC_CAL2
- U12 pad 95: VDD_3V3 -> VDD_3V3_MCU
- U12 pad 99: Net-(U12-Pad99) -> SWEN
- U13 pad 12: ENCSCK1 -> GPEX_SCK
- U13 pad 13: ENCMOSI1 -> GPEX_MOSI
- U13 pad 14: ENCMISO1 -> GPEX_MISO
- U13 pad 15: Net-(R43-Pad1) -> GND
- U13 pad 16: Net-(R44-Pad1) -> GND
- U13 pad 17: Net-(R45-Pad1) -> GND
- U15 pad 1: Net-(U11-Pad2) -> Net-(TP56-Pad1)
- U15 pad 4: Net-(U11-Pad1) -> Net-(TP57-Pad1)
- U17 pad 1: Net-(U17-Pad1) -> GND
- U17 pad 2: Net-(U17-Pad2) -> GND
- U17 pad 3: Net-(U17-Pad3) -> GND
- U18 pad 5: USB_5V -> Net-(J1-Pad1)
- U19 pad 1: Net-(C45-Pad1) -> Net-(C169-Pad1)
- U19 pad 6: USB_5V -> Net-(C52-Pad1)
- U19 pad 7: Net-(TP18-Pad1) -> Net-(R35-Pad2)
- U19 pad 8: Net-(C45-Pad1) -> Net-(C169-Pad1)
- U21 pad 20: Net-(R63-Pad2) -> GND
- U21 pad 21: Net-(R64-Pad2) -> GND
- U22 pad 1: Net-(R61-Pad1) -> USB_5V
- U23 pad 12: ENCSG1 -> PWM_IN1
- U23 pad 17: ENCSY1 -> Net-(D15-Pad1)
- U23 pad 22: VDD_3V3 -> VDD_3V3_MCU
- U23 pad 23: Net-(R66-Pad1) -> USB_5V
- U23 pad 7: ENCIRQ1 -> MOTOR1_BRKIN
- U24 pad 12: ENCSG2 -> PWM_IN2
- U24 pad 17: ENCSY2 -> Net-(D33-Pad1)
- U24 pad 22: VDD_3V3 -> VDD_3V3_MCU
- U24 pad 23: Net-(R67-Pad1) -> USB_5V
- U24 pad 3: ENCMISO1 -> ENCMISO2
- U24 pad 5: ENCSCK1 -> ENCSCK2
- U24 pad 6: ENCMOSI1 -> ENCMOSI2
- U26 pad 1: Net-(R76-Pad2) -> VMOT_SENSE
- U26 pad 10: Net-(R90-Pad1) -> Net-(R205-Pad1)
- U26 pad 12: Net-(R94-Pad1) -> Net-(R207-Pad1)
- U26 pad 13: Net-(R111-Pad2) -> Net-(U26-Pad13)
- U26 pad 14: Net-(R111-Pad1) -> Net-(U26-Pad13)
- U26 pad 2: Net-(R76-Pad2) -> VMOT_SENSE
- U26 pad 5: Net-(R88-Pad1) -> Net-(R203-Pad1)
- U26 pad 6: Net-(R132-Pad1) -> Net-(U26-Pad6)
- U26 pad 7: Net-(R132-Pad1) -> Net-(U26-Pad6)
- U26 pad 8: Net-(R135-Pad1) -> Net-(U26-Pad8)
- U26 pad 9: Net-(R135-Pad1) -> Net-(U26-Pad8)
- U27 pad 1: SOB1 -> SOA1
- U27 pad 3: SOA1 -> SOB1
- U27 pad 4: Net-(R80-Pad2) -> Net-(R81-Pad2)
- U27 pad 5: VDD_3V3 -> VDD_3V3_MCU
- U27 pad 6: Net-(R81-Pad2) -> Net-(R80-Pad2)
- U28 pad 1: SOB2 -> SOA2
- U28 pad 3: SOA2 -> SOB2
- U28 pad 4: Net-(R82-Pad2) -> Net-(R83-Pad2)
- U28 pad 5: VDD_3V3 -> VDD_3V3_MCU
- U28 pad 6: Net-(R83-Pad2) -> Net-(R82-Pad2)
- U29 pad 10: GND -> VDD_3V3
- U29 pad 8: VDD_3V3 -> GND
- U3 pad 4: AIN_VDD_5V -> USB_5V
- U30 pad 18: ECAT_SYNC1 -> Net-(TP102-Pad1)
- U30 pad 34: ECAT_SYNC0 -> Net-(TP101-Pad1)
- U31 pad 29: Net-(C100-Pad1) -> VMOT
- U32 pad 11: OC_ADJ1 -> OC_ADJ2
- U32 pad 29: Net-(C101-Pad1) -> VMOT
- U33 pad 1: Net-(R112-Pad1) -> Net-(R132-Pad1)
- U33 pad 10: Net-(R134-Pad1) -> Net-(R131-Pad1)
- U33 pad 2: Net-(R112-Pad2) -> Net-(R132-Pad1)
- U33 pad 3: Net-(R97-Pad1) -> Net-(R88-Pad1)
- U33 pad 5: Net-(R131-Pad1) -> Net-(R94-Pad1)
- U33 pad 6: Net-(R133-Pad1) -> Net-(R111-Pad2)
- U33 pad 7: Net-(R153-Pad1) -> VSA1
- U33 pad 8: Net-(R154-Pad1) -> VSB1
- U33 pad 9: Net-(R136-Pad1) -> Net-(R133-Pad1)
- U34 pad 1: Net-(R109-Pad2) -> GND
- U34 pad 2: Net-(R109-Pad2) -> GND
- U34 pad 3: Net-(R109-Pad2) -> GND
- U35 pad 1: VSC2 -> Net-(R135-Pad1)
- U35 pad 10: (no net) -> Net-(R134-Pad1)
- U35 pad 12: (no net) -> Net-(R180-Pad1)
- U35 pad 13: (no net) -> Net-(R182-Pad1)
- U35 pad 14: (no net) -> VSC2
- U35 pad 2: Net-(R182-Pad1) -> Net-(R135-Pad1)
- U35 pad 3: Net-(R180-Pad1) -> Net-(R90-Pad1)
- U35 pad 5: (no net) -> Net-(R97-Pad1)
- U35 pad 6: (no net) -> Net-(R112-Pad2)
- U35 pad 7: (no net) -> VSA2
- U35 pad 8: (no net) -> VSB2
- U35 pad 9: (no net) -> Net-(R136-Pad1)
- U36 pad 1: PWM_IN1 -> USB_5V
- U36 pad 2: VDD_3V3 -> GND
- U36 pad 3: PWM_IN2 -> Net-(R67-Pad1)
- U36 pad 5: Net-(U36-Pad5) -> Net-(C152-Pad1)
- U4 pad 4: AIN_VDD_5V -> USB_5V
- U5 pad 12: ENCSCK1 -> GPIO_SCK
- U5 pad 13: ENCMOSI1 -> GPIO_MOSI
- U5 pad 14: ENCMISO1 -> GPIO_MISO
- U5 pad 15: Net-(R34-Pad1) -> GND
- U5 pad 16: Net-(R35-Pad1) -> GND
- U5 pad 17: Net-(R36-Pad1) -> GND
- U6 pad 10: POTADDR2 -> POTADDRB
- U6 pad 6: Net-(U6-Pad6) -> GND
- U6 pad 9: POTADDR3 -> POTADDRC
- U7 pad 2: Net-(C16-Pad1) -> VREF1
- U8 pad 8: CAN_STB1 -> GND
- U9 pad 8: CAN_STB2 -> GND
Other:
- copper layers 2 -> 4

Commit message: pcb layout
Parts:
- moved TP67 20.2 mm to (91.2, 12.0), turned to 270 degrees
- moved TP70 18.7 mm to (92.2, 12.0), turned to 270 degrees
- moved TP69 18.0 mm to (93.2, 12.0), turned to 270 degrees
- moved TP72 16.3 mm to (94.2, 12.0), turned to 270 degrees
- moved TP68 16.1 mm to (96.2, 12.0), turned to 270 degrees
- moved TP71 15.5 mm to (95.2, 12.0), turned to 270 degrees
- moved C120 5.55 mm to (110.8, -14.0)
- moved R129 5.55 mm to (113.0, -8.25)
- moved R130 5.55 mm to (113.0, -10.2)
- moved TP87 5.55 mm to (114.0, -8.25)
- moved TP88 5.55 mm to (114.0, -10.2)
- moved U34 5.55 mm to (108.5, -10.5)
- moved D18 0.56 mm to (115.5, -13.0)
- moved TP101 0.25 mm to (103.2, -0.50)

Commit message: optimize connector size
Parts:
- removed C158, C51: CAP_2.2uF_16V_0402, Capacitor_SMD:C_0402_1005Metric
- removed P10, P12: CONN_SENSOR, CUSTOM:CONN_SENSOR
- removed P29, P30, P31, P32, P33, P34, P35, P36: CONN_LED, CUSTOM:CONN_LED
- added R214: RES_NOFIT_0402, Resistor_SMD:R_0402_1005Metric, F.Cu at (77.8, -125.8)
- added R215: RES_NOFIT_0402, Resistor_SMD:R_0402_1005Metric, F.Cu at (113.6, -127.2)
- added R216: RES_NOFIT_0402, Resistor_SMD:R_0402_1005Metric, F.Cu at (103.5, -137.2)
- added R217: RES_NOFIT_0402, Resistor_SMD:R_0402_1005Metric, F.Cu at (100.5, -137.2)
- added R218: RES_NOFIT_0402, Resistor_SMD:R_0402_1005Metric, F.Cu at (100.0, -125.8)
- added R219: RES_NOFIT_0402, Resistor_SMD:R_0402_1005Metric, F.Cu at (103.2, -125.8)
- added R220: RES_NOFIT_0402, Resistor_SMD:R_0402_1005Metric, F.Cu at (82.2, -137.2)
- added R221: RES_NOFIT_0402, Resistor_SMD:R_0402_1005Metric, F.Cu at (79.2, -137.2)
- added R222: RES_NOFIT_0402, Resistor_SMD:R_0402_1005Metric, F.Cu at (78.8, -125.8)
- added R223: RES_NOFIT_0402, Resistor_SMD:R_0402_1005Metric, F.Cu at (82.2, -125.8)
- added R224: RES_NOFIT_0402, Resistor_SMD:R_0402_1005Metric, F.Cu at (113.8, -136.5)
- added R225: RES_NOFIT_0402, Resistor_SMD:R_0402_1005Metric, F.Cu at (104.5, -137.2)
- added R226: RES_NOFIT_0402, Resistor_SMD:R_0402_1005Metric, F.Cu at (97.5, -137.2)
- added R227: RES_NOFIT_0402, Resistor_SMD:R_0402_1005Metric, F.Cu at (99.0, -125.8)
- added R228: RES_NOFIT_0402, Resistor_SMD:R_0402_1005Metric, F.Cu at (106.2, -125.8)
- added R229: RES_NOFIT_0402, Resistor_SMD:R_0402_1005Metric, F.Cu at (83.2, -137.2)
- added R230: RES_NOFIT_0402, Resistor_SMD:R_0402_1005Metric, F.Cu at (78.2, -137.2)
- added R231: RES_NOFIT_0402, Resistor_SMD:R_0402_1005Metric, F.Cu at (83.2, -125.8)
- added R232: RES_NOFIT_0402, Resistor_SMD:R_0402_1005Metric, F.Cu at (262.7, 53.8)
- added R233: RES_NOFIT_0402, Resistor_SMD:R_0402_1005Metric, F.Cu at (264.4, 52.8)
- added R234: RES_NOFIT_0402, Resistor_SMD:R_0402_1005Metric, F.Cu at (261.0, 51.8)
- added R235: RES_NOFIT_0402, Resistor_SMD:R_0402_1005Metric, F.Cu at (259.3, 50.8)
- added R236: RES_NOFIT_0402, Resistor_SMD:R_0402_1005Metric, F.Cu at (257.6, 51.8)
- added R237: RES_NOFIT_0402, Resistor_SMD:R_0402_1005Metric, F.Cu at (259.3, 49.8)
- added R238: RES_NOFIT_0402, Resistor_SMD:R_0402_1005Metric, F.Cu at (257.6, 50.8)
- P1, P2, P3, P4, P5, P6, P7, P8: value CONN_SWITCH -> CONN_BUTTON; footprint CUSTOM:CONN_SWITCH -> CUSTOM:CONN_BUTTON
- P11, P9: value CONN_SENSOR -> CONN_JOYSTICK; footprint CUSTOM:CONN_SENSOR -> CUSTOM:CONN_JOYSTICK
- R34: value RES_10K_1%_0402 -> RES_NOFIT_0402
- moved P49 358.8 mm to (189.5, -201.8), turned to 180 degrees
- moved P2 321.6 mm to (146.2, -206.5), turned to 180 degrees
- moved C49 321.0 mm to (118.2, -190.5)
- moved P46 316.1 mm to (70.5, -186.2), turned to 270 degrees
- moved C57 315.9 mm to (113.8, -194.2), turned to 90 degrees
- moved TP64 314.6 mm to (90.2, -126.8), turned to 270 degrees
- moved P1 313.6 mm to (158.5, -206.5), turned to 180 degrees
- moved C53 313.3 mm to (115.5, -191.0), turned to 180 degrees
- moved C163 312.8 mm to (73.5, -113.4), turned to 270 degrees
- moved TP65 311.7 mm to (89.2, -126.8), turned to 270 degrees
- moved P6 310.1 mm to (97.1, -206.5), turned to 180 degrees
- moved TP63 309.2 mm to (91.2, -126.8), turned to 270 degrees
- moved P7 308.0 mm to (84.8, -206.5), turned to 180 degrees
- moved C56 307.5 mm to (113.8, -192.5), turned to 270 degrees
- moved C162 305.3 mm to (86.2, -113.4), turned to 270 degrees
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Connections:
- P1 pad 1: Net-(P1-Pad1) -> GND
- P1 pad 2: GND -> SW_IN1
- P11 pad 2: Net-(P11-Pad2) -> GND
- P11 pad 3: GND -> Net-(P11-Pad3)
- P2 pad 1: Net-(P2-Pad1) -> GND
- P2 pad 2: GND -> SW_IN2
- P3 pad 1: Net-(P3-Pad1) -> GND
- P3 pad 2: GND -> SW_IN3
- P4 pad 1: Net-(P4-Pad1) -> GND
- P4 pad 2: GND -> SW_IN4
- P5 pad 1: Net-(P5-Pad1) -> GND
- P5 pad 2: GND -> SW_IN5
- P6 pad 1: Net-(P6-Pad1) -> GND
- P6 pad 2: GND -> SW_IN6
- P7 pad 1: Net-(P7-Pad1) -> GND
- P7 pad 2: GND -> SW_IN7
- P8 pad 1: Net-(P8-Pad1) -> GND
- P8 pad 2: GND -> SW_IN8
- P9 pad 2: Net-(P9-Pad2) -> GND
- P9 pad 3: GND -> Net-(P9-Pad3)
- R2 pad 2: Net-(P9-Pad2) -> Net-(P9-Pad3)
- R3 pad 2: Net-(P10-Pad2) -> Net-(P9-Pad4)
- R4 pad 2: Net-(P11-Pad2) -> Net-(P11-Pad3)
- R5 pad 2: Net-(P12-Pad2) -> Net-(P11-Pad4)
- U2 pad 2: Net-(P1-Pad1) -> SW_IN1
- U2 pad 3: Net-(P2-Pad1) -> SW_IN2
- U2 pad 4: Net-(P3-Pad1) -> SW_IN3
- U2 pad 5: Net-(P4-Pad1) -> SW_IN4
- U2 pad 6: Net-(P5-Pad1) -> SW_IN5
- U2 pad 7: Net-(P6-Pad1) -> SW_IN6
- U2 pad 8: Net-(P7-Pad1) -> SW_IN7
- U2 pad 9: Net-(P8-Pad1) -> SW_IN8
- U21 pad 12: Net-(P29-Pad1) -> LED_OUT8
- U21 pad 13: Net-(P30-Pad1) -> LED_OUT7
- U21 pad 14: Net-(P31-Pad1) -> LED_OUT6
- U21 pad 15: Net-(P32-Pad1) -> LED_OUT5
- U21 pad 16: Net-(P33-Pad1) -> LED_OUT4
- U21 pad 17: Net-(P34-Pad1) -> LED_OUT3
- U21 pad 18: Net-(P35-Pad1) -> LED_OUT2
- U21 pad 19: Net-(P36-Pad1) -> LED_OUT1

Commit message: place second motor driver
Parts:
- moved TP97 393.3 mm to (-96.8, -48.8)
- moved R166 345.8 mm to (56.0, -200.5), turned to 270 degrees
- moved TP34 339.6 mm to (-96.8, -43.8)
- moved TP36 338.9 mm to (-96.8, -42.8)
- moved R52 336.7 mm to (198.5, -202.5), turned to 90 degrees
- moved C147 336.4 mm to (48.8, -200.5), turned to 270 degrees
- moved TP32 333.0 mm to (-96.8, -44.8)
- moved R112 332.4 mm to (-88.2, -58.0)
- moved R164 332.2 mm to (59.5, -200.5), turned to 270 degrees
- moved R194 331.7 mm to (-78.8, -65.0), turned to 180 degrees
- moved C98 330.8 mm to (-88.2, -62.0)
- moved R188 328.9 mm to (53.5, -200.5), turned to 270 degrees
- moved C92 328.8 mm to (-89.0, -43.8), turned to 180 degrees
- moved TP30 328.5 mm to (-96.8, -45.8)
- moved R187 327.4 mm to (57.0, -200.5), turned to 270 degrees
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
Commit message: review footprints and horizontal vertical stuff
Parts:
- P37, P41: value CONN_ENCODER -> ENCODER; footprint TerminalBlock_4Ucon:TerminalBlock_4Ucon_1x08_P3.50mm_Horizontal -> CUSTOM:CONN_ENCODER
- moved D33 546.5 mm to (43.4, -377.8), turned to 180 degrees
- moved C60 533.4 mm to (46.8, -382.4)
- moved C62 518.0 mm to (46.8, -383.4)
- moved R74 514.6 mm to (73.8, -369.4), turned to 270 degrees
- moved C68 511.5 mm to (74.8, -369.4), turned to 90 degrees
- moved R73 508.9 mm to (66.8, -369.4), turned to 90 degrees
- moved C79 504.4 mm to (42.4, -370.2), turned to 270 degrees
- moved C77 499.7 mm to (87.8, -369.4), turned to 270 degrees
- moved C80 492.3 mm to (54.6, -370.2), turned to 270 degrees
- moved C78 487.2 mm to (29.8, -370.2), turned to 90 degrees
- moved U24 483.3 mm to (42.8, -382.0)
- moved R75 475.7 mm to (80.8, -369.4), turned to 90 degrees
- moved C67 474.7 mm to (67.8, -369.4), turned to 270 degrees
- moved C69 473.9 mm to (81.8, -369.4), turned to 270 degrees
- moved C81 442.0 mm to (147.6, -302.2), turned to 90 degrees
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Other:
- board text added: "MOTOR 1"
- board text added: "MOTOR 2"
- board text added: "Supply Sense"
