File: motordriver-2x.kicad_sch (KiCad schematic)
At the start: 672 parts, among them J1 USB_B_Micro, J2 CONN_RJ45_MAG, J3 CONN_RJ45_MAG, P1 CONN_BUTTON, P11 CONN_JOYSTICK, P13 CONN_SENSOR, P14 CONN_SENSOR, P15 CONN_SENSOR, P16 CONN_SENSOR, P17 CONN_DEBUG_2R, P18 CONN_POWER_41A, P19 CONN_CAN, P2 CONN_BUTTON, P20 CONN_CAN, P21 CONN_AN_OUT, P22 CONN_AN_OUT, P23 CONN_POWER_10A, P24 CONN_CAN, P25 CONN_LCD, P26 CONN_AN_OUT, P27 CONN_AN_OUT, P28 CONN_UEXT, P3 CONN_BUTTON, P37 CONN_ENCODER, P38 CONN_SENSOR, P39 CONN_SENSOR, P4 CONN_BUTTON, P40 CONN_SENSOR, P41 CONN_ENCODER, P42 CONN_SENSOR, P43 CONN_SENSOR, P44 CONN_SENSOR, P45 CONN_MOTOR, P46 CONN_MOTOR, P47 CONN_HALL, P48 CONN_HALL, P49 CONN_BRKRES, P5 CONN_BUTTON, P6 CONN_BUTTON, P7 CONN_BUTTON, P8 CONN_BUTTON, P9 CONN_JOYSTICK, Q1 Q_NMOS_2X_60V_63A, Q2 Q_NMOS_2X_60V_63A, Q3 Q_NMOS_2X_60V_63A, Q4 Q_NMOS_2X_60V_63A, Q5 Q_NMOS_2X_60V_63A, Q6 Q_NMOS_2X_60V_63A, Q7 Q_PNP_BC856, Q8 Q_NMOS_BUK9875, U1 IC_MIC2026, U10 IC_MCP4461, U11 IC_MCP2517FD-xJHA, U12 IC_STM32F429ZET6, U13 IC_MCP23S17, U14 IC_TPS54360DDA, U15 IC_TJA1044GT3, U16 IC_TLV2474, U17 IC_M24C16, U18 IC_USBLC6-2, U19 IC_TPS62147RGXR, U2 IC_MAX6818, U20 IC_TLV75533, U21 IC_LP55231, U22 IC_TLV75533, U23 IC_MAX14890, U24 IC_MAX14890, U25 IC_MIC2026, U26 IC_TLV2474, U27 IC_USBLC6-2, U28 IC_USBLC6-2, U29 IC_MCP4461, U3 IC_TLV2474, U30 IC_LAN9252, U31 IC_DRV8302, U32 IC_DRV8302, U33 IC_TLV2474, U34 IC_M24C16, U35 IC_TLV2474, U36 IC_TLV75533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

Commit message: bom: add bom generation
Closes #4

Signed-off-by: Martin Schröder <info@swedishembedded.com>
Parts:
- D10, D11, D13: MPN ESDCAN03-2BWY -> ESDCAN03-2BWY
- D31: Datasheet_1 (none) -> https://www.mouser.com/datasheet/2/348/sml-d15(c)-e-1508222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
- Q8: MPN BUK9875-100A/CUX -> BUK9875-100A/CUX
- R10, R11, R12, R13, R14, R15, R16, R17, R65: Datasheet_1 (none) -> https://www.mouser.com/datasheet/2/427/dcrcwe3-109170.pdf
- R101, R102, R105, R106, R138, R139, R142, R143, R170, R171, R174, R175: renamed from ?; Datasheet_1 (none) -> https://www.mouser.com/datasheet/2/315/AOA0000C304-1149620.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
- R111, R112, R153, R154, R163, R164, R165, R166, R167, R168, R193, R194: renamed from ?; MPN RC0402FR-075KL -> RC0402FR-075KL
- R147, R148: renamed from ?; Datasheet_1 (none) -> https://www.mouser.com/datasheet/2/427/dcrcwe3-109170.pdf
- R198: renamed from ?; Datasheet_1 (none) -> https://www.mouser.com/datasheet/2/427/crcwce3-1223726.pdf
- R46, R47, R56, R57, R69: MPN RC0402FR-075KL -> RC0402FR-075KL
- R50: Datasheet_1 (none) -> https://www.mouser.com/datasheet/2/427/crcwce3-1223726.pdf
- R51, R52: Datasheet_1 (none) -> https://www.mouser.com/datasheet/2/315/AOA0000C304-1149620.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
- S2: Datasheet_1 (none) -> https://www.mouser.com/datasheet/2/307/en-a6h-1221378.pdf
- gave numbers to parts that had none: 301
